Commit message: Better URDF Robot

File: src/gazebo/Master_ASM/urdf/Master_ASM.urdf (robot description, URDF)
Before this commit: robot Master_ASM, 3 links, 2 joints
Links:
- removed link SwerveL
- removed link WheelsL
- added link swerve1_Link, mass 2.5211; visual mesh filename=package://Master_ASM/meshes/swerve1_Link.STL
- added link swerve2_Link, mass 2.5211; visual mesh filename=package://Master_ASM/meshes/swerve2_Link.STL
- added link swerve3_Link, mass 2.5211; visual mesh filename=package://Master_ASM/meshes/swerve3_Link.STL
- added link swerve4_Link, mass 2.5211; visual mesh filename=package://Master_ASM/meshes/swerve4_Link.STL
- added link wheel1_Link, mass 1.1372; visual mesh filename=package://Master_ASM/meshes/wheel1_Link.STL
- added link wheel2_Link, mass 1.1372; visual mesh filename=package://Master_ASM/meshes/wheel2_Link.STL
- added link wheel3_Link, mass 1.1372; visual mesh filename=package://Master_ASM/meshes/wheel3_Link.STL
- added link wheel4_Link, mass 1.1372; visual mesh filename=package://Master_ASM/meshes/wheel4_Link.STL
- link base_link: mass 38.0385728398503 -> 38.039
Joints:
- removed joint Swerve
- removed joint Wheels
- added joint swerve1_joint: type continuous, parent base_link, child swerve1_Link, origin xyz=-0.34701 0.55026 -0.59563 rpy=1.5708 0 0, axis 0 0 1
- added joint swerve2_joint: type continuous, parent base_link, child swerve2_Link, origin xyz=0.34701 -0.55026 -0.59563 rpy=1.5708 0 3.1416, axis 0 1 0
- added joint swerve3_joint: type continuous, parent base_link, child swerve3_Link, origin xyz=0.34701 0.55014 -0.59563 rpy=1.5708 0 3.1416, axis 0 0 1
- added joint swerve4_joint: type continuous, parent base_link, child swerve4_Link, origin xyz=-0.34701 -0.55014 -0.59563 rpy=1.5708 0 0, axis 0 0 1
- added joint wheel1_joint: type continuous, parent swerve1_Link, child wheel1_Link, origin xyz=0.071447 0.038959 0.1082 rpy=1.5708 0.34561 1.5708, axis 0 0 1
- added joint wheel2_joint: type continuous, parent swerve2_Link, child wheel2_Link, origin xyz=0.071447 0.038959 0.1082 rpy=1.5708 0.34561 1.5708, axis 0 0 1
- added joint wheel3_joint: type continuous, parent swerve3_Link, child wheel3_Link, origin xyz=0.071447 0.038959 0.1082 rpy=1.5708 0.34561 1.5708, axis 0 0 1
- added joint wheel4_joint: type continuous, parent swerve4_Link, child wheel4_Link, origin xyz=0.071447 0.038959 0.1082 rpy=1.5708 0.34561 1.5708, axis 0 0 1

Commit message: basic movement

File: src/gazebo/Master_ASM/urdf/Master_ASM.urdf (robot description, URDF)
Before this commit: robot Master_ASM, 9 links, 8 joints
Links:
- link base_link: geometry collision box size=0.73 1.4 0.6; visual mesh filename=package://Master_ASM/meshes/base_link.STL
- link swerve1_Link: geometry visual box size=0.1 0.2 0.1
- link swerve2_Link: geometry visual box size=0.1 0.2 0.1
- link swerve3_Link: geometry visual box size=0.1 0.2 0.1
- link swerve4_Link: geometry visual box size=0.1 0.2 0.1
- link wheel1_Link: geometry collision mesh filename=package://Master_ASM/meshes/wheel1_Link.STL; visual mesh filename=package://Master_ASM/meshes/wheel1_Link.STL
- link wheel2_Link: geometry collision mesh filename=package://Master_ASM/meshes/wheel2_Link.STL; visual mesh filename=package://Master_ASM/meshes/wheel2_Link.STL
- link wheel3_Link: geometry collision mesh filename=package://Master_ASM/meshes/wheel3_Link.STL; visual mesh filename=package://Master_ASM/meshes/wheel3_Link.STL
- link wheel4_Link: geometry collision mesh filename=package://Master_ASM/meshes/wheel4_Link.STL; visual mesh filename=package://Master_ASM/meshes/wheel4_Link.STL
Joints:
- joint swerve1_joint: axis 0 0 1 -> 0 1 0; type continuous -> fixed
- joint swerve2_joint: type continuous -> fixed
- joint swerve3_joint: axis 0 0 1 -> 0 1 0; type continuous -> fixed
- joint swerve4_joint: axis 0 0 1 -> 0 1 0; type continuous -> fixed
- joint wheel1_joint: axis 0 0 1 -> 0 0 -1; origin xyz=0.071447 0.038959 0.1082 rpy=1.5708 0.34561 1.5708 -> xyz=0 0 0 rpy=1.5708 0.34561 1.5708
- joint wheel2_joint: origin xyz=0.071447 0.038959 0.1082 rpy=1.5708 0.34561 1.5708 -> xyz=0 0 0 rpy=1.5708 0.34561 1.5708
- joint wheel3_joint: origin xyz=0.071447 0.038959 0.1082 rpy=1.5708 0.34561 1.5708 -> xyz=0 0 0 rpy=1.5708 0.34561 1.5708
- joint wheel4_joint: axis 0 0 1 -> 0 0 -1; origin xyz=0.071447 0.038959 0.1082 rpy=1.5708 0.34561 1.5708 -> xyz=0 0 0 rpy=1.5708 0.34561 1.5708

Commit message: robot works?

File: src/gazebo/Master_ASM/urdf/Master_ASM.urdf (robot description, URDF)
Before this commit: robot Master_ASM, 9 links, 8 joints
Links:
- link wheel1_Link: geometry collision cylinder length=0.2 radius=0.115; visual mesh filename=package://Master_ASM/meshes/wheel1_Link.STL
- link wheel2_Link: geometry collision cylinder length=0.2 radius=0.115; visual mesh filename=package://Master_ASM/meshes/wheel2_Link.STL
- link wheel3_Link: geometry collision cylinder length=0.2 radius=0.115; visual mesh filename=package://Master_ASM/meshes/wheel3_Link.STL
- link wheel4_Link: geometry collision cylinder length=0.2 radius=0.115; visual mesh filename=package://Master_ASM/meshes/wheel4_Link.STL
Joints:
- joint swerve1_joint: type fixed -> continuous
- joint swerve2_joint: type fixed -> continuous
- joint swerve3_joint: type fixed -> continuous
- joint swerve4_joint: type fixed -> continuous
