Commit message: remove unneeded stl files

File: src/gazebo/ros_gz_description/models/master_ASM/urdf/master_ASM.urdf (robot description, URDF)
Before this commit: robot Master_ASM, 9 links, 8 joints
Links:
- link wheel1_Link: geometry collision cylinder length=0.2 radius=0.115; visual mesh filename=../meshes/wheel_Link.STL
- link wheel2_Link: geometry collision cylinder length=0.2 radius=0.115; visual mesh filename=../meshes/wheel_Link.STL
- link wheel3_Link: geometry collision cylinder length=0.2 radius=0.115; visual mesh filename=../meshes/wheel_Link.STL
- link wheel4_Link: geometry collision cylinder length=0.2 radius=0.115; visual mesh filename=../meshes/wheel_Link.STL

Commit message: depth and camera box correct size

File: src/gazebo/ros_gz_description/models/master_ASM/urdf/master_ASM.urdf (robot description, URDF)
Before this commit: robot Master_ASM, 10 links, 9 joints
Links:
- link camera_link: geometry visual box size=0.03025 0.17525 0.04310
Joints:
- joint camera_joint: origin xyz=0.305 0 0.08 rpy=0 0 0 -> xyz=0.35 0 0.05 rpy=0 0 0
