Commit message: Seperate robot state publishers from gazebo Add seperate pacakge called robot_description which contains a robot_state_publisher This reduces code duplication overall if it need to be used on actual robot

File: src/robot_description/models/master_ASM/urdf/master_ASM.urdf (robot description, URDF)
Before this commit: robot Master_ASM, 10 links, 9 joints
Links:
- link base_link: geometry collision box size=0.7317 1.4254 0.6435; visual mesh filename=package://robot_description/models/master_ASM/meshes/base_l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
- link camera_link: geometry collision mesh filename=package://robot_description/models/master_ASM/meshes/zed2i.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; visual mesh filename=package://robot_description/models/master_ASM/meshes/zed2i.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
- link wheel1_Link: geometry collision cylinder length=0.2 radius=0.115; visual mesh filename=package://robot_description/models/master_ASM/meshes/wheel_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
- link wheel2_Link: geometry collision cylinder length=0.2 radius=0.115; visual mesh filename=package://robot_description/models/master_ASM/meshes/wheel_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
- link wheel3_Link: geometry collision cylinder length=0.2 radius=0.115; visual mesh filename=package://robot_description/models/master_ASM/meshes/wheel_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
- link wheel4_Link: geometry collision cylinder length=0.2 radius=0.115; visual mesh filename=package://robot_description/models/master_ASM/meshes/wheel_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

Commit message: Utilize zed xarco in robot description

File: src/robot_description/models/master_ASM/urdf/master_ASM.urdf (robot description, URDF)
Before this commit: robot Master_ASM, 10 links, 9 joints
Links:
- removed link camera_link
- added link zed2i_camera_center; collision mesh filename=package://zed_interfaces/meshes/zed2i.stl; visual mesh filename=package://zed_interfaces/meshes/zed2i.stl
- added link zed2i_camera_link
- added link zed2i_left_camera_frame
- added link zed2i_left_camera_optical_frame
- added link zed2i_right_camera_frame
- added link zed2i_right_camera_optical_frame
Joints:
- added joint zed2i_camera_center_joint: type fixed, parent zed2i_camera_link, child zed2i_camera_center, origin xyz=0 0 0.015 rpy=0 0.0 0
- added joint zed2i_left_camera_joint: type fixed, parent zed2i_camera_center, child zed2i_left_camera_frame, origin xyz=-0.01 0.06 0 rpy=0 0 0
- added joint zed2i_left_camera_optical_joint: type fixed, parent zed2i_left_camera_frame, child zed2i_left_camera_optical_frame, origin xyz=0 0 0 rpy=-1.5707963267948966 0.0 -1.5707963267948966
- added joint zed2i_right_camera_joint: type fixed, parent zed2i_camera_center, child zed2i_right_camera_frame, origin xyz=-0.01 -0.06 0 rpy=0 0 0
- added joint zed2i_right_camera_optical_joint: type fixed, parent zed2i_right_camera_frame, child zed2i_right_camera_optical_frame, origin xyz=0 0 0 rpy=-1.5707963267948966 0.0 -1.5707963267948966
- joint camera_joint: child camera_link -> zed2i_camera_link; origin xyz=0.343 0.009 -0.1254 rpy=0 0.52359878 0 -> xyz=0.343 0.009 -0.1254 rpy=0 2.5 3.14

Commit message: Fix base_link

File: src/robot_description/models/master_ASM/urdf/master_ASM.urdf (robot description, URDF)
Before this commit: robot Master_ASM, 15 links, 14 joints
Joints:
- joint camera_joint: child zed2i_camera_link -> base_link; origin xyz=0.343 0.009 -0.1254 rpy=0 2.5 3.14 -> xyz=-0.343 -0.009 -0.1254 rpy=0 -0.52359878 0; parent base_link -> zed2i_camera_link

Commit message: Initial working changes

File: src/robot_description/models/master_ASM/urdf/master_ASM.urdf (robot description, URDF)
Before this commit: robot Master_ASM, 15 links, 14 joints
Joints:
- joint camera_joint: child base_link -> zed2i_camera_link; origin xyz=-0.343 -0.009 -0.1254 rpy=0 -0.52359878 0 -> xyz=0.343 -0.009 -0.1254 rpy=0 0.52359878 0; parent zed2i_camera_link -> base_link

File: src/robot_description/models/master_ASM/urdf/master_ASM.urdf.xacro (robot description, xacro)
@@ -48,7 +48,7 @@
   </xacro:zed_camera>
   <joint name="camera_joint" type="fixed">
-    <child link="base_link"/>
-    <parent link="zed2i_camera_link"/>
-    <origin xyz="-0.343 -0.009 -0.1254" rpy="0 -0.52359878 0" />
+    <parent link="base_link"/>
+    <child link="zed2i_camera_link"/>
+    <origin xyz="0.343 -0.009 -0.1254" rpy="0 0.52359878 0" />
   </joint>
   <gazebo reference="zed2i_camera_link">

Commit message: current working state

File: src/robot_description/models/master_ASM/urdf/master_ASM.urdf (robot description, URDF)
Before this commit: robot Master_ASM, 15 links, 14 joints
Joints:
- joint camera_joint: origin xyz=-0.343 -0.009 -0.1254 rpy=0 -0.52359878 0 -> xyz=-0.343 -0.009 -0.1254 rpy=0 0 0

File: src/robot_description/models/master_ASM/urdf/master_ASM.urdf.xacro (robot description, xacro)
@@ -50,5 +50,5 @@
     <child link="base_link"/>
     <parent link="zed2i_camera_link"/>
-    <origin xyz="-0.343 -0.009 -0.1254" rpy="0 -0.52359878 0" />
+    <origin xyz="-0.343 -0.009 -0.1254" rpy="0 0 0" /> <!-- TODO: we are not actually mounting the ZED parallel to the ground -->
   </joint>
   <gazebo reference="zed2i_camera_link">

Commit message: improvements

File: src/robot_description/models/master_ASM/urdf/master_ASM.urdf (robot description, URDF)
Before this commit: robot Master_ASM, 15 links, 14 joints
Joints:
- joint camera_joint: origin xyz=-0.343 -0.009 -0.1254 rpy=0 0 0 -> xyz=-0.343 -0.009 -0.1254 rpy=0 -0.52359878 0

File: src/robot_description/models/master_ASM/urdf/master_ASM.urdf.xacro (robot description, xacro)
@@ -50,5 +50,5 @@
     <child link="base_link"/>
     <parent link="zed2i_camera_link"/>
-    <origin xyz="-0.343 -0.009 -0.1254" rpy="0 0 0" /> <!-- TODO: we are not actually mounting the ZED parallel to the ground -->
+    <origin xyz="-0.343 -0.009 -0.1254" rpy="0 -0.52359878 0" />
   </joint>
   <gazebo reference="zed2i_camera_link">

Commit message: bring back translation_end _vector for easier accurate positioning

File: src/robot_description/models/master_ASM/urdf/master_ASM.urdf (robot description, URDF)
Before this commit: robot Master_ASM, 15 links, 14 joints
Links:
- added link translation_end_link, mass 0.001
Joints:
- removed joint camera_joint
- added joint camera_to_translation_end: type fixed, parent zed2i_camera_link, child translation_end_link, origin xyz=0 0 0 rpy=0 -0.52359878 0
- added joint translation_end_to_base: type fixed, parent translation_end_link, child base_link, origin xyz=-0.343 -0.009 0.1254 rpy=0 0 0

File: src/robot_description/models/master_ASM/urdf/master_ASM.urdf.xacro (robot description, xacro)
@@ -44,11 +44,26 @@
     </collision>
   </link>
+  <!-- Connect the base_link to the new link with only a translation -->
+  <joint name="translation_end_to_base" type="fixed">
+    <parent link="translation_end_link"/>
+    <child link="base_link"/>
+    <origin xyz="-0.343 -0.009 0.1254" rpy="0 0 0"/>
+  </joint>
+  <!-- Add a new link at the end of the translation vector -->
+  <link name="translation_end_link">
+    <inertial>
+      <origin xyz="0 0 0" rpy="0 0 0"/>
+      <mass value="0.001"/>
+      <inertia ixx="0.0001" ixy="0" ixz="0" iyy="0.0001" iyz="0" izz="0.0001"/>
+    </inertial>
+  </link>
+  <!-- Connect the new link to the camera_link with only a rotation -->
   <xacro:include filename="$(find zed_wrapper)/urdf/zed_macro.urdf.xacro" />
   <xacro:zed_camera name="zed2i" model="zed2i">
   </xacro:zed_camera>
-  <joint name="camera_joint" type="fixed">
-    <child link="base_link"/>
+  <joint name="camera_to_translation_end" type="fixed">
     <parent link="zed2i_camera_link"/>
-    <origin xyz="-0.343 -0.009 -0.1254" rpy="0 -0.52359878 0" />
+    <child link="translation_end_link"/>
+    <origin xyz="0 0 0" rpy="0 -0.52359878 0"/>
   </joint>
   <gazebo reference="zed2i_camera_link">

Commit message: Refactor to reduce code duplication across sim vs real robot

File: src/robot_description/models/master_ASM/urdf/master_ASM.urdf (robot description, URDF)
Before this commit: robot Master_ASM, 15 links, 14 joints
Joints:
- joint camera_joint: origin xyz=0.343 -0.009 -0.1254 rpy=0 0.52359878 0 -> xyz=0.343 -0.009 -0.1254 rpy=0 0 0
