Commit message: Update robot.urdf.xacro dimensions

File: src/robot_description/models/master_ASM/urdf/robot.urdf.xacro (robot description, xacro)
@@ -1,11 +1,15 @@
 <?xml version="1.0" encoding="utf-8"?>
 <robot name="robot_base" xmlns:xacro="http://www.ros.org/wiki/xacro">
-    <xacro:property name="chassisHeight" value="0.64"/>
+    <xacro:property name="chassisHeight" value="0.57476257962"/>
     <xacro:property name="chassisLength" value="1.1"/>
-    <xacro:property name="chassisWidth" value="0.512"/>
+    <xacro:property name="chassisWidth" value="0.5077"/>
     <xacro:property name="chassisMass" value="55"/>
     <xacro:property name="wheelWidth" value="0.11"/>
-    <xacro:property name="wheelRadius" value="0.15"/>
+    <xacro:property name="wheelRadius" value="0.16"/>
     <xacro:property name="wheelMass" value="2"/>
+    <!-- Distance between middle - middle front back wheels 0.873175 m -->
+    <!-- Distance between middle - middle Left and right wheels 0.62285 m -->
+    <!-- Distance from back of chassis to middle of back wheels 0.1534125 -->
+    <!-- Distance from bottem of chassis to middle of wheels 0.0475 (below) -->
     <xacro:property name="pretty" value="true"/>
     <material name="grey">

Commit message: Update robot.urdf.xacro more

File: src/robot_description/models/master_ASM/urdf/robot.urdf.xacro (robot description, xacro)
@@ -1,6 +1,6 @@
 <?xml version="1.0" encoding="utf-8"?>
 <robot name="robot_base" xmlns:xacro="http://www.ros.org/wiki/xacro">
-    <xacro:property name="chassisHeight" value="0.57476257962"/>
-    <xacro:property name="chassisLength" value="1.1"/>
+    <xacro:property name="chassisHeight" value="0.66976"/>
+    <xacro:property name="chassisLength" value="1.13198"/>
     <xacro:property name="chassisWidth" value="0.5077"/>
     <xacro:property name="chassisMass" value="55"/>
@@ -11,5 +11,5 @@
     <!-- Distance between middle - middle Left and right wheels 0.62285 m -->
     <!-- Distance from back of chassis to middle of back wheels 0.1534125 -->
-    <!-- Distance from bottem of chassis to middle of wheels 0.0475 (below) -->
+    <!-- Distance from bottom of chassis to middle of wheels 0.11789257822 -->
     <xacro:property name="pretty" value="true"/>
     <material name="grey">
