Commit message: using macros now

File: src/robot_description/models/master_ASM/urdf/macros.urdf.xacro (robot description, xacro)
@@ -1,4 +1,50 @@
 <?xml version="1.0" encoding="utf-8"?>
-<robot name="macros" xmlns:xacro="http://www.ros.org/wiki/xacro">
-<xacro:macro name="wheel" params="name">
+<robot xmlns:xacro="http://www.ros.org/wiki/xacro">
+<xacro:macro name="wheel_link" params="name pretty:=^|true wheelRadius:=^ wheelWidth:=^ wheelMass:=^ *origin">
+    <link name="${name}">
+        <inertial>
+            <xacro:insert_block name="origin" />
+            <mass value="${wheelMass}" />
+            <inertia
+                ixx="0.0059462"
+                ixy="0"
+                ixz="0"
+                iyy="0.0059468"
+                iyz="0"
+                izz="0.0072591" />
+        </inertial>
+        <visual>
+            <xacro:insert_block name="origin" />
+            <geometry>
+            <xacro:if value="${pretty}">
+                <mesh
+                filename="$(find robot_description)/models/master_ASM/meshes/wheel_Link.STL" />
+            </xacro:if>
+            <xacro:unless value="${pretty}">
+                <cylinder radius="${wheelRadius}" length="${wheelWidth}" />
+            </xacro:unless>
+            </geometry>
+            <material name="grey" />
+        </visual>
+        <collision>
+            <xacro:insert_block name="origin" />
+            <geometry>
+                <cylinder radius="${wheelRadius}" length="${wheelWidth}" />
+            </geometry>
+        </collision>
+    </link>
 </xacro:macro>
+<xacro:macro name="wheel_joint" params="wheel x y z">
+    <joint
+        name="${str(wheel) + '_joint'}"
+        type="continuous">
+        <origin
+            xyz="${x} ${y} -${z}"
+            rpy="${pi/2} 0 ${pi/2}" />
+        <parent link="frame_link" />
+        <child link="${str(wheel) + '_link'}" />
+        <axis
+        xyz="0 0 -1" />
+    </joint>
+</xacro:macro>
+</robot>

File: src/robot_description/models/master_ASM/urdf/master_ASM.urdf.xacro (robot description, xacro)
@@ -4,5 +4,6 @@
      Commit Version: 1.6.0-4-g7f85cfe  Build Version: 1.6.7995.38578
      For more information, please see http://wiki.ros.org/sw_urdf_exporter -->
-<robot name="Complicated" xmlns:xacro="http://www.ros.org/wiki/xacro">
+<robot name="master_ASM" xmlns:xacro="http://www.ros.org/wiki/xacro">
+  <xacro:include filename="robot.urdf.xacro" />
   <link name="base_link">
     <origin xyz="0 0 0" rpy="0 0 0" />
@@ -11,45 +12,6 @@
     <parent link="base_link" />
     <child link="frame_link" />
-    <origin xyz="0 0 0" rpy="0 0 -1.5708" />
+    <origin xyz="0 0 0" rpy="0 0 ${-pi/2}" />
   </joint>
-  <link
-    name="frame_link">
-    <inertial>
-      <origin
-        xyz="0.0012829 -0.31468 -0.0059364"
-        rpy="0 0 0" />
-      <mass
-        value="38.039" />
-      <inertia
-        ixx="0.51975"
-        ixy="0.00069908"
-        ixz="2.9544E-06"
-        iyy="0.93889"
-        iyz="-3.8081E-06"
-        izz="0.5273" />
-    </inertial>
-    <visual>
-      <origin
-        xyz="0 0 0"
-        rpy="0 0 0" />
-      <geometry>
-        <mesh
-          filename="package://robot_description/models/master_ASM/meshes/frame_link.STL" />
-      </geometry>
-      <material
-        name="">
-        <color
-          rgba="0.79216 0.81961 0.93333 1" />
-      </material>
-    </visual>
-    <collision>
-      <origin
-        xyz="0 0 -0.2"
-        rpy="0 0 0" />
-      <geometry>
-        <box size="0.7317 1.4254 0.6435" />
-      </geometry>
-    </collision>
-  </link>
   <!-- ZED 2i Camera -->
   <!-- <xacro:arg name="use_zed_localization" default="true" />
@@ -118,418 +80,34 @@
     </sensor>
   </gazebo>
-  <link
-    name="swerve1_Link">
-    <inertial>
-      <origin
-        xyz="0.072878 0.028694 7.0574E-06"
-        rpy="0 0 0" />
-      <mass
-        value="2.5211" />
-      <inertia
-        ixx="0.008233"
-        ixy="5.8978E-05"
-        ixz="5.7912E-08"
-        iyy="0.006818"
-        iyz="1.2459E-07"
-        izz="0.0069443" />
-    </inertial>
-    <visual>
-      <origin
-        xyz="0 0 0"
-        rpy="0 0 0" />
-      <geometry>
-        <box size="0.1 0.2 0.1" />
-      </geometry>
-      <material
-        name="">
-        <color
-          rgba="0.75294 0.75294 0.75294 1" />
-      </material>
-    </visual>
-  </link>
-  <joint
-    name="swerve1_joint"
-    type="fixed">
-    <origin
-      xyz="-0.34701 0.55026 -0.59563"
-      rpy="1.5708 0 0" />
-    <parent
-      link="frame_link" />
-    <child
-      link="swerve1_Link" />
-    <axis
-      xyz="0 1 0" />
-    <!-- <limit lower="6.28" upper="6.28" effort="30" velocity="1.0" /> -->
-  </joint>
-  <link
-    name="wheel1_Link">
-    <inertial>
-      <origin
-        xyz="2.9097E-09 -0.115 -0.00055956"
-        rpy="0 0 0" />
-      <mass
-        value="1.1372" />
-      <inertia
-        ixx="0.0059462"
-        ixy="1.6529E-09"
-        ixz="-6.3363E-10"
-        iyy="0.0059468"
-        iyz="6.9163E-09"
-        izz="0.0072591" />
-    </inertial>
-    <visual>
-      <origin
-        xyz="0 0.115 0"
-        rpy="0 0 0" />
-      <geometry>
-        <mesh
-          filename="package://robot_description/models/master_ASM/meshes/wheel_Link.STL" />
-      </geometry>
-      <material
-        name="">
-        <color
-          rgba="0.79216 0.81961 0.93333 1" />
-      </material>
-    </visual>
-    <collision>
-      <origin
-        xyz="0 0 0"
-        rpy="0 0 0" />
-      <geometry>
-        <cylinder radius="0.115" length="0.2" />
-      </geometry>
-    </collision>
-  </link>
-  <joint
-    name="wheel1_joint"
-    type="continuous">
-    <origin
-      xyz="0 0 0"
-      rpy="1.5708 0.34561 1.5708" />
-    <parent
-      link="swerve1_Link" />
-    <child
-      link="wheel1_Link" />
-    <axis
-      xyz="0 0 -1" />
-  </joint>
-  <link
-    name="swerve2_Link">
-    <inertial>
-      <origin
-        xyz="0.072878 0.028694 7.0574E-06"
-        rpy="0 0 0" />
-      <mass
-        value="2.5211" />
-      <inertia
-        ixx="0.008233"
-        ixy="5.8978E-05"
-        ixz="5.7912E-08"
-        iyy="0.006818"
-        iyz="1.2459E-07"
-        izz="0.0069443" />
-    </inertial>
-    <visual>
-      <origin
-        xyz="0 0 0"
-        rpy="0 0 0" />
-      <geometry>
-        <box size="0.1 0.2 0.1" />
-      </geometry>
-      <material
-        name="">
-        <color
-          rgba="0.75294 0.75294 0.75294 1" />
-      </material>
-    </visual>
-  </link>
-  <joint
-    name="swerve2_joint"
-    type="fixed">
-    <origin
-      xyz="0.34701 -0.55026 -0.59563"
-      rpy="1.5708 0 3.1416" />
-    <parent
-      link="frame_link" />
-    <child
-      link="swerve2_Link" />
-    <axis
-      xyz="0 1 0" />
-    <!-- <limit lower="6.28" upper="6.28" effort="30" velocity="1.0" /> -->
-  </joint>
-  <link
-    name="wheel2_Link">
-    <inertial>
-      <origin
-        xyz="2.9097E-09 -0.115 -0.00055956"
-        rpy="0 0 0" />
-      <mass
-        value="1.1372" />
-      <inertia
-        ixx="0.0059462"
-        ixy="1.6529E-09"
-        ixz="-6.3363E-10"
-        iyy="0.0059468"
-        iyz="6.9163E-09"
-        izz="0.0072591" />
-    </inertial>
-    <visual>
-      <origin
-        xyz="0 0.115 0"
-        rpy="0 0 0" />
-      <geometry>
-        <mesh
-          filename="package://robot_description/models/master_ASM/meshes/wheel_Link.STL" />
-      </geometry>
-      <material
-        name="">
-        <color
-          rgba="0.79216 0.81961 0.93333 1" />
-      </material>
-    </visual>
-    <collision>
-      <origin
-        xyz="0 0 0"
-        rpy="0 0 0" />
-      <geometry>
-        <!-- <mesh
-          filename="package://Master_ASM/meshes/wheel2_Link.STL" /> -->
-        <cylinder radius="0.115" length="0.2" />
-      </geometry>
-    </collision>
-  </link>
-  <joint
-    name="wheel2_joint"
-    type="continuous">
-    <origin
-      xyz="0 0 0"
-      rpy="1.5708 0.34561 1.5708" />
-    <parent
-      link="swerve2_Link" />
-    <child
-      link="wheel2_Link" />
-    <axis
-      xyz="0 0 1" />
-  </joint>
-  <link
-    name="swerve3_Link">
-    <inertial>
-      <origin
-        xyz="0.072878 0.028694 7.0574E-06"
-        rpy="0 0 0" />
-      <mass
-        value="2.5211" />
-      <inertia
-        ixx="0.008233"
-        ixy="5.8978E-05"
-        ixz="5.7912E-08"
-        iyy="0.006818"
-        iyz="1.2459E-07"
-        izz="0.0069443" />
-    </inertial>
-    <visual>
-      <origin
-        xyz="0 0 0"
-        rpy="0 0 0" />
-      <geometry>
-        <box size="0.1 0.2 0.1" />
-      </geometry>
-      <material
-        name="">
-        <color
-          rgba="0.75294 0.75294 0.75294 1" />
-      </material>
-    </visual>
-  </link>
-  <joint
-    name="swerve3_joint"
-    type="fixed">
-    <origin
-      xyz="0.34701 0.55014 -0.59563"
-      rpy="1.5708 0 3.1416" />
-    <parent
-      link="frame_link" />
-    <child
-      link="swerve3_Link" />
-    <axis
-      xyz="0 1 0" />
-  </joint>
-  <link
-    name="wheel3_Link">
-    <inertial>
-      <origin
-        xyz="2.9097E-09 -0.115 -0.00055956"
-        rpy="0 0 0" />
-      <mass
-        value="1.1372" />
-      <inertia
-        ixx="0.0059462"
-        ixy="1.6529E-09"
-        ixz="-6.3363E-10"
-        iyy="0.0059468"
-        iyz="6.9163E-09"
-        izz="0.0072591" />
-    </inertial>
-    <visual>
-      <origin
-        xyz="0 0.115 0"
-        rpy="0 0 0" />
-      <geometry>
-        <mesh
-          filename="package://robot_description/models/master_ASM/meshes/wheel_Link.STL" />
-      </geometry>
-      <material
-        name="">
-        <color
-          rgba="0.79216 0.81961 0.93333 1" />
-      </material>
-    </visual>
-    <collision>
-      <origin
-        xyz="0 0 0"
-        rpy="0 0 0" />
-      <geometry>
-        <cylinder radius="0.115" length="0.2" />
-      </geometry>
-    </collision>
-  </link>
-  <joint
-    name="wheel3_joint"
-    type="continuous">
-    <origin
-      xyz="0 0 0"
-      rpy="1.5708 0.34561 1.5708" />
-    <parent
-      link="swerve3_Link" />
-    <child
-      link="wheel3_Link" />
-    <axis
-      xyz="0 0 1" />
-  </joint>
-  <link
-    name="swerve4_Link">
-    <inertial>
-      <origin
-        xyz="0.072878 0.028694 7.0574E-06"
-        rpy="0 0 0" />
-      <mass
-        value="2.5211" />
-      <inertia
-        ixx="0.008233"
-        ixy="5.8978E-05"
-        ixz="5.7912E-08"
-        iyy="0.006818"
-        iyz="1.2459E-07"
-        izz="0.0069443" />
-    </inertial>
-    <visual>
-      <origin
-        xyz="0 0 0"
-        rpy="0 0 0" />
-      <geometry>
-        <box size="0.1 0.2 0.1" />
-      </geometry>
-      <material
-        name="">
-        <color
-          rgba="0.75294 0.75294 0.75294 1" />
-      </material>
-    </visual>
-  </link>
-  <joint
-    name="swerve4_joint"
-    type="fixed">
-    <origin
-      xyz="-0.34701 -0.55014 -0.59563"
-      rpy="1.5708 0 0" />
-    <parent
-      link="frame_link" />
-    <child
-      link="swerve4_Link" />
-    <axis
-      xyz="0 1 0" />
-  </joint>
-  <link
-    name="wheel4_Link">
-    <inertial>
-      <origin
-        xyz="2.9097E-09 -0.115 -0.00055956"
-        rpy="0 0 0" />
-      <mass
-        value="1.1372" />
-      <inertia
-        ixx="0.0059462"
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
File: src/robot_description/models/master_ASM/urdf/robot.urdf.xacro (robot description, xacro)
@@ -1,4 +1,4 @@
 <?xml version="1.0" encoding="utf-8"?>
-<robot name="robot" xmlns:xacro="http://www.ros.org/wiki/xacro">
+<robot name="robot_base" xmlns:xacro="http://www.ros.org/wiki/xacro">
     <xacro:property name="chassisHeight" value="0.64"/>
     <xacro:property name="chassisLength" value="1.1"/>
@@ -9,13 +9,9 @@
     <xacro:property name="wheelMass" value="2"/>
     <xacro:property name="pretty" value="true"/>
+    <material name="grey">
+        <color
+        rgba="0.79216 0.81961 0.93333 1" />
+    </material>
     <xacro:include filename="macros.urdf.xacro" />
-    <link name="base_link">
-        <origin xyz="0 0 0" rpy="0 0 0" />
-    </link>
-    <joint name="base_to_frame_joint" type="fixed">
-        <parent link="base_link" />
-        <child link="frame_link" />
-        <origin xyz="0 0 0" rpy="0 0 -1.5708" />
-    </joint>
     <link name="frame_link">
         <inertial>
@@ -41,47 +37,5 @@
             </xacro:unless>
         </geometry>
-        <material
-            name="">
-            <color
-            rgba="0.79216 0.81961 0.93333 1" />
-        </material>
-        </visual>
-        <collision>
-        <origin
-            xyz="0 0 -0.2"
-            rpy="0 0 0" />
-        <geometry>
-            <box size="0.7317 1.4254 0.6435" />
-        </geometry>
-        </collision>
-    </link>
-    <link name="wheel1_Link">
-        <inertial>
-        <origin
-            xyz="0 -0.115 0"
-            rpy="0 0 0" />
-        <mass
-            value="1.1372" />
-        <inertia
-            ixx="0.0059462"
-            ixy="0"
-            ixz="0"
-            iyy="0.0059468"
-            iyz="0"
-            izz="0.0072591" />
-        </inertial>
-        <visual>
-        <origin
-            xyz="0 0.115 0"
-            rpy="0 0 0" />
-        <geometry>
-            <mesh
-            filename="package://robot_description/models/master_ASM/meshes/wheel_Link.STL" />
-        </geometry>
-        <material
-            name="">
-            <color
-            rgba="0.79216 0.81961 0.93333 1" />
-        </material>
+        <material name="grey" />
         </visual>
         <collision>
@@ -90,202 +44,23 @@
             rpy="0 0 0" />
         <geometry>
-            <cylinder radius="0.115" length="0.2" />
+            <box size="${chassisWidth} ${chassisLength} ${chassisHeight}"/>
         </geometry>
         </collision>
     </link>
-    <joint
-        name="wheel1_joint"
-        type="continuous">
-        <origin
-        xyz="0 0 0"
-        rpy="1.5708 0.34561 1.5708" />
-        <parent link="frame_link" />
-        <child link="wheel1_Link" />
-        <axis
-        xyz="0 0 -1" />
-    </joint>
-    <link name="wheel2_Link">
-        <inertial>
-        <origin
-            xyz="0 -0.115 0"
-            rpy="0 0 0" />
-        <mass
-            value="1.1372" />
-        <inertia
-            ixx="0.0059462"
-            ixy="0"
-            ixz="0"
-            iyy="0.0059468"
-            iyz="0"
-            izz="0.0072591" />
-        </inertial>
-        <visual>
-        <origin
-            xyz="0 0.115 0"
-            rpy="0 0 0" />
-        <geometry>
-            <mesh
-            filename="package://robot_description/models/master_ASM/meshes/wheel_Link.STL" />
-        </geometry>
-        <material
-            name="">
-            <color
-            rgba="0.79216 0.81961 0.93333 1" />
-        </material>
-        </visual>
-        <collision>
-        <origin
-            xyz="0 0 0"
-            rpy="0 0 0" />
-        <geometry>
-            <!-- <mesh
-            filename="package://Master_ASM/meshes/wheel2_Link.STL" /> -->
-            <cylinder radius="0.115" length="0.2" />
-        </geometry>
-        </collision>
-    </link>
-    <joint name="wheel2_joint"
-        type="continuous">
-        <origin
-        xyz="0 0 0"
-        rpy="1.5708 0.34561 1.5708" />
-        <parent
-        link="frame_link" />
-        <child
-        link="wheel2_Link" />
-        <axis
-        xyz="0 0 1" />
-    </joint>
-    <link name="wheel3_Link">
-        <inertial>
-        <origin
-            xyz="0 -0.115 0"
-            rpy="0 0 0" />
-        <mass
-            value= "${wheelMass}" />
-        <inertia
-            ixx="0.0059462"
-            ixy="0"
-            ixz="0"
-            iyy="0.0059468"
-            iyz="0"
-            izz="0.0072591" />
-        </inertial>
-        <visual>
-        <origin
-            xyz="0 0.115 0"
-            rpy="0 0 0" />
-        <geometry>
-            <mesh
-            filename="package://robot_description/models/master_ASM/meshes/wheel_Link.STL" />
-        </geometry>
-        <material
-            name="">
-            <color
-            rgba="0.79216 0.81961 0.93333 1" />
-        </material>
-        </visual>
-        <collision>
-        <origin
-            xyz="0 0 0"
-            rpy="0 0 0" />
-        <geometry>
-            <cylinder radius="0.115" length="0.2" />
-        </geometry>
-        </collision>
-    </link>
-    <joint
-        name="wheel3_joint"
-        type="continuous">
-        <origin
-        xyz="0 0 0"
-        rpy="1.5708 0.34561 1.5708" />
-        <parent
-        link="frame_link" />
-        <child
-        link="wheel3_Link" />
-        <axis
-        xyz="0 0 1" />
-    </joint>
-    <link name="wheel4_Link">
-        <inertial>
-        <origin
-            xyz="2.9097E-09 -0.115 -0.00055956"
-            rpy="0 0 0" />
-        <mass
-            value="1.1372" />
-        <inertia
-            ixx="0.0059462"
-            ixy="1.6529E-09"
-            ixz="-6.3363E-10"
-            iyy="0.0059468"
-            iyz="6.9163E-09"
-            izz="0.0072591" />
-        </inertial>
-        <visual>
-        <origin
-            xyz="0 0.115 0"
-            rpy="0 0 0" />
-        <geometry>
-            <mesh
-            filename="package://robot_description/models/master_ASM/meshes/wheel_Link.STL" />
-        </geometry>
-        <material
-            name="">
-            <color
-            rgba="0.79216 0.81961 0.93333 1" />
-        </material>
-        </visual>
-        <collision>
-        <origin
-            xyz="0 0 0"
-            rpy="0 0 0" />
-        <geometry>
-            <cylinder radius="0.115" length="0.2" />
-        </geometry>
-        </collision>
-    </link>
-    <joint name="wheel4_joint"
-        type="continuous">
-        <origin
-        xyz="0 0 0"
-        rpy="1.5708 0.34561 1.5708" />
-        <parent
-        link="frame_link" />
-        <child
-        link="wheel4_Link" />
-        <axis
-        xyz="0 0 -1" />
-    </joint>
-    <gazebo>
-        <plugin
-        filename="ignition-gazebo-joint-state-publisher-system"
-        name="ignition::gazebo::systems::JointStatePublisher">
-        <topic>joint_states</topic>
-        </plugin>
-        <plugin
-        filename="ignition-gazebo-joint-controller-system"
-        name="ignition::gazebo::systems::JointController">
-        <joint_name>wheel1_joint</joint_name>
-        <initial_velocity>0.0</initial_velocity>
-        </plugin>
-        <plugin
-        filename="ignition-gazebo-joint-controller-system"
-        name="ignition::gazebo::systems::JointController">
-        <joint_name>wheel2_joint</joint_name>
-        <initial_velocity>0.0</initial_velocity>
-        </plugin>
-        <plugin
-        filename="ignition-gazebo-joint-controller-system"
-        name="ignition::gazebo::systems::JointController">
-        <joint_name>wheel3_joint</joint_name>
-        <initial_velocity>0.0</initial_velocity>
-        </plugin>
-        <plugin
-        filename="ignition-gazebo-joint-controller-system"
-        name="ignition::gazebo::systems::JointController">
-        <joint_name>wheel4_joint</joint_name>
-        <initial_velocity>0.0</initial_velocity>
-        </plugin>
-    </gazebo>
+    <xacro:wheel_link name="wheel1_link">
+        <origin xyz="0 0 0" rpy="0 0 0" />
+    </xacro:wheel_link>
+    <xacro:wheel_joint wheel="wheel1" x="${chassisWidth/2+wheelWidth/3}" y="${chassisLength/2}" z="${chassisHeight/2}"/>
+    <xacro:wheel_link name="wheel2_link">
+        <origin xyz="0 0 0" rpy="0 0 0" />
+    </xacro:wheel_link>
+    <xacro:wheel_joint wheel="wheel2" x="${chassisWidth/2+wheelWidth/3}" y="-${chassisLength/2}" z="${chassisHeight/2}"/>
+    <xacro:wheel_link name="wheel3_link">
+        <origin xyz="0 0 0" rpy="0 0 0" />
+    </xacro:wheel_link>
+    <xacro:wheel_joint wheel="wheel3" x="-${chassisWidth/2+wheelWidth/3}" y="-${chassisLength/2}" z="${chassisHeight/2}"/>
+    <xacro:wheel_link name="wheel4_link">
+        <origin xyz="0 0 0" rpy="0 0 0" />
+    </xacro:wheel_link>
+    <xacro:wheel_joint wheel="wheel4" x="-${chassisWidth/2+wheelWidth/3}" y="${chassisLength/2}" z="${chassisHeight/2}"/>
 </robot>
