Commit message: zed xacro

File: src/robot_description/models/master_ASM/urdf/macros.urdf.xacro (robot description, xacro)
@@ -1,8 +1,8 @@
 <?xml version="1.0" encoding="utf-8"?>
 <robot xmlns:xacro="http://www.ros.org/wiki/xacro">
-<xacro:macro name="wheel_link" params="name pretty:=^|true wheelRadius:=^ wheelWidth:=^ wheelMass:=^ *origin">
+<xacro:macro name="wheel_link" params="name pretty:=^|true wheelRadius:=^ wheelWidth:=^ wheelMass:=^">
     <link name="${name}">
         <inertial>
-            <xacro:insert_block name="origin" />
+            <origin xyz="0 0 0" rpy="0 0 0" />
             <mass value="${wheelMass}" />
             <inertia
@@ -15,5 +15,5 @@
         </inertial>
         <visual>
-            <xacro:insert_block name="origin" />
+            <origin xyz="0 0 0" rpy="0 0 0" />
             <geometry>
             <xacro:if value="${pretty}">
@@ -28,5 +28,5 @@
         </visual>
         <collision>
-            <xacro:insert_block name="origin" />
+            <origin xyz="0 0 0" rpy="0 0 0" />
             <geometry>
                 <cylinder radius="${wheelRadius}" length="${wheelWidth}" />

File: src/robot_description/models/master_ASM/urdf/master_ASM.urdf.xacro (robot description, xacro)
@@ -15,27 +15,5 @@
   </joint>
   <!-- ZED 2i Camera -->
-  <!-- <xacro:arg name="use_zed_localization" default="true" />
-  <xacro:include filename="$(find zed_wrapper)/urdf/zed_macro.urdf.xacro" />
-  <xacro:zed_camera name="zed2i" model="zed2i" enable_gnss="false"> -->
-    <!-- This block is required even if enable_gnss="false" for some reason, but you can leave it empty -->
-    <!-- <gnss_origin></gnss_origin>
-  </xacro:zed_camera> -->
-  <!-- Add a joint to connect the ZED 2i Camera model to the robot -->
-  <!-- <xacro:if value="$(arg use_zed_localization)"> -->
-    <!-- ZED Localization -> The reference link is 'zed2i_camera_link' and 'base_link' is a child -->
-    <!-- <joint name="zed2i_joint" type="fixed">
-      <parent link="zed2i_camera_link"/>
-      <child link="base_link"/>
-      <origin xyz="-0.5 0 0.375" rpy="0 0 0"/>
-    </joint>
-  </xacro:if>
-  <xacro:unless value="$(arg use_zed_localization)"> -->
-    <!-- NO ZED Localization -> 'zed2i_camera_link' is a child of 'base_link' -->
-    <!-- <joint name="zed2i_joint" type="fixed">
-      <parent link="base_link"/>
-      <child link="zed2i_camera_link"/>
-      <origin xyz="0.5 0 -0.375" rpy="0 0 0"/>
-    </joint>
-  </xacro:unless> -->
+  <xacro:include filename="zed.urdf.xacro" />
   <gazebo reference="zed2i_camera_link">
     <sensor name="camera" type="camera">
@@ -90,5 +68,5 @@
         name="ignition::gazebo::systems::JointController">
         <joint_name>wheel1_joint</joint_name>
-        <initial_velocity>0.0</initial_velocity>
+        <initial_velocity>1.0</initial_velocity>
         </plugin>
         <plugin
@@ -96,5 +74,5 @@
         name="ignition::gazebo::systems::JointController">
         <joint_name>wheel2_joint</joint_name>
-        <initial_velocity>0.0</initial_velocity>
+        <initial_velocity>1.0</initial_velocity>
         </plugin>
         <plugin
@@ -102,5 +80,5 @@
         name="ignition::gazebo::systems::JointController">
         <joint_name>wheel3_joint</joint_name>
-        <initial_velocity>0.0</initial_velocity>
+        <initial_velocity>1.0</initial_velocity>
         </plugin>
         <plugin
@@ -108,5 +86,5 @@
         name="ignition::gazebo::systems::JointController">
         <joint_name>wheel4_joint</joint_name>
-        <initial_velocity>0.0</initial_velocity>
+        <initial_velocity>1.0</initial_velocity>
         </plugin>
     </gazebo>

File: src/robot_description/models/master_ASM/urdf/robot.urdf.xacro (robot description, xacro)
@@ -48,19 +48,11 @@
         </collision>
     </link>
-    <xacro:wheel_link name="wheel1_link">
-        <origin xyz="0 0 0" rpy="0 0 0" />
-    </xacro:wheel_link>
+    <xacro:wheel_link name="wheel1_link" />
     <xacro:wheel_joint wheel="wheel1" x="${chassisWidth/2+wheelWidth/3}" y="${chassisLength/2}" z="${chassisHeight/2}"/>
-    <xacro:wheel_link name="wheel2_link">
-        <origin xyz="0 0 0" rpy="0 0 0" />
-    </xacro:wheel_link>
+    <xacro:wheel_link name="wheel2_link" />
     <xacro:wheel_joint wheel="wheel2" x="${chassisWidth/2+wheelWidth/3}" y="-${chassisLength/2}" z="${chassisHeight/2}"/>
-    <xacro:wheel_link name="wheel3_link">
-        <origin xyz="0 0 0" rpy="0 0 0" />
-    </xacro:wheel_link>
+    <xacro:wheel_link name="wheel3_link" />
     <xacro:wheel_joint wheel="wheel3" x="-${chassisWidth/2+wheelWidth/3}" y="-${chassisLength/2}" z="${chassisHeight/2}"/>
-    <xacro:wheel_link name="wheel4_link">
-        <origin xyz="0 0 0" rpy="0 0 0" />
-    </xacro:wheel_link>
+    <xacro:wheel_link name="wheel4_link" />
     <xacro:wheel_joint wheel="wheel4" x="-${chassisWidth/2+wheelWidth/3}" y="${chassisLength/2}" z="${chassisHeight/2}"/>
 </robot>

Commit message: new measurements and wheel placements

File: src/robot_description/models/master_ASM/urdf/macros.urdf.xacro (robot description, xacro)
@@ -19,5 +19,5 @@
             <xacro:if value="${pretty}">
                 <mesh
-                filename="$(find robot_description)/models/master_ASM/meshes/wheel_Link.STL" />
+                filename="../meshes/ASM_Drive_Assembly.STL" scale="0.001 0.001 0.001"/> <!-- stl is measured in mm, need m -->
             </xacro:if>
             <xacro:unless value="${pretty}">

File: src/robot_description/models/master_ASM/urdf/master_ASM.urdf.xacro (robot description, xacro)
@@ -67,5 +67,5 @@
         filename="ignition-gazebo-joint-controller-system"
         name="ignition::gazebo::systems::JointController">
-        <joint_name>wheel1_joint</joint_name>
+        <joint_name>wheelFrontLeft_joint</joint_name>
         <initial_velocity>1.0</initial_velocity>
         </plugin>
@@ -73,5 +73,5 @@
         filename="ignition-gazebo-joint-controller-system"
         name="ignition::gazebo::systems::JointController">
-        <joint_name>wheel2_joint</joint_name>
+        <joint_name>wheelFrontRight_joint</joint_name>
         <initial_velocity>1.0</initial_velocity>
         </plugin>
@@ -79,5 +79,5 @@
         filename="ignition-gazebo-joint-controller-system"
         name="ignition::gazebo::systems::JointController">
-        <joint_name>wheel3_joint</joint_name>
+        <joint_name>wheelBackLeft_joint</joint_name>
         <initial_velocity>1.0</initial_velocity>
         </plugin>
@@ -85,5 +85,5 @@
         filename="ignition-gazebo-joint-controller-system"
         name="ignition::gazebo::systems::JointController">
-        <joint_name>wheel4_joint</joint_name>
+        <joint_name>wheelBackRight_joint</joint_name>
         <initial_velocity>1.0</initial_velocity>
         </plugin>

File: src/robot_description/models/master_ASM/urdf/robot.urdf.xacro (robot description, xacro)
@@ -9,8 +9,12 @@
     <xacro:property name="wheelMass" value="2"/>
     <!-- Distance between middle - middle front back wheels 0.873175 m -->
-    <!-- Distance between middle - middle Left and right wheels 0.62285 m -->
+    <!-- Distance between middle - middle Left and right wheels 0.62285 m --> <!-- double check, bad mesaurement to middle of wheel -->
     <!-- Distance from back of chassis to middle of back wheels 0.1534125 -->
-    <!-- Distance from bottom of chassis to middle of wheels 0.11789257822 -->
-    <xacro:property name="pretty" value="true"/>
+    <!-- Distance from bottom of chassis to middle of wheels 0.0475 -->
+    <xacro:property name="wheelDeltaWidth" value="${(chassisWidth + wheelWidth)/2}" />
+    <xacro:property name="wheelDeltaBack" value="${-1 * (chassisLength/2 - 0.1534125)}" />
+    <xacro:property name="wheelDeltaFront" value="${wheelDeltaBack + 0.873175}" />
+    <xacro:property name="wheelDeltaHeight" value="${(chassisHeight/2 - 0.0475)}" />
+    <xacro:property name="pretty" value="false"/>
     <material name="grey">
         <color
@@ -35,5 +39,5 @@
             <xacro:if value="${pretty}">
                 <mesh
-                filename="package://robot_description/models/master_ASM/meshes/frame_link.STL" />
+                filename="../meshes/chassis.STL" scale="0.001 0.001 0.001"/> <!-- stl is measured in mm, need m -->
             </xacro:if>
             <xacro:unless value="${pretty}">
@@ -52,11 +56,11 @@
         </collision>
     </link>
-    <xacro:wheel_link name="wheel1_link" />
-    <xacro:wheel_joint wheel="wheel1" x="${chassisWidth/2+wheelWidth/3}" y="${chassisLength/2}" z="${chassisHeight/2}"/>
-    <xacro:wheel_link name="wheel2_link" />
-    <xacro:wheel_joint wheel="wheel2" x="${chassisWidth/2+wheelWidth/3}" y="-${chassisLength/2}" z="${chassisHeight/2}"/>
-    <xacro:wheel_link name="wheel3_link" />
-    <xacro:wheel_joint wheel="wheel3" x="-${chassisWidth/2+wheelWidth/3}" y="-${chassisLength/2}" z="${chassisHeight/2}"/>
-    <xacro:wheel_link name="wheel4_link" />
-    <xacro:wheel_joint wheel="wheel4" x="-${chassisWidth/2+wheelWidth/3}" y="${chassisLength/2}" z="${chassisHeight/2}"/>
+    <xacro:wheel_link name="wheelFrontLeft_link" />
+    <xacro:wheel_joint wheel="wheelFrontLeft" x="-${wheelDeltaWidth}" y="${wheelDeltaFront}" z="${wheelDeltaHeight}"/>
+    <xacro:wheel_link name="wheelFrontRight_link" />
+    <xacro:wheel_joint wheel="wheelFrontRight" x="${wheelDeltaWidth}" y="${wheelDeltaFront}" z="${wheelDeltaHeight}"/>
+    <xacro:wheel_link name="wheelBackLeft_link" />
+    <xacro:wheel_joint wheel="wheelBackLeft" x="-${wheelDeltaWidth}" y="${wheelDeltaBack}" z="${wheelDeltaHeight}"/>
+    <xacro:wheel_link name="wheelBackRight_link" />
+    <xacro:wheel_joint wheel="wheelBackRight" x="${wheelDeltaWidth}" y="${wheelDeltaBack}" z="${wheelDeltaHeight}"/>
 </robot>

Commit message: figured out where that bug was

File: src/robot_description/models/master_ASM/urdf/macros.urdf.xacro (robot description, xacro)
@@ -40,5 +40,5 @@
         type="continuous">
         <origin
-            xyz="${x} ${y} -${z}"
+            xyz="${x} ${y} ${z}"
             rpy="${pi/2} 0 ${pi/2}" />
         <parent link="frame_link" />

File: src/robot_description/models/master_ASM/urdf/robot.urdf.xacro (robot description, xacro)
@@ -13,7 +13,7 @@
     <!-- Distance from bottom of chassis to middle of wheels 0.0475 -->
     <xacro:property name="wheelDeltaWidth" value="${(chassisWidth + wheelWidth)/2}" />
-    <xacro:property name="wheelDeltaBack" value="${-1 * (chassisLength/2 - 0.1534125)}" />
+    <xacro:property name="wheelDeltaBack" value="-${chassisLength/2 - 0.1534125}" />
     <xacro:property name="wheelDeltaFront" value="${wheelDeltaBack + 0.873175}" />
-    <xacro:property name="wheelDeltaHeight" value="${(chassisHeight/2 - 0.0475)}" />
+    <xacro:property name="wheelDeltaHeight" value="-${chassisHeight/2 - 0.0475}" />
     <xacro:property name="pretty" value="false"/>
     <material name="grey">

Commit message: wheel name changes and degugging

File: src/robot_description/models/master_ASM/urdf/macros.urdf.xacro (robot description, xacro)
@@ -1,16 +1,21 @@
 <?xml version="1.0" encoding="utf-8"?>
 <robot xmlns:xacro="http://www.ros.org/wiki/xacro">
+<xacro:macro name="box_inertia" params="m x y z">
+    <mass value="${m}" />
+    <inertia  ixx="${m*(y*y+z*z)/12}" ixy = "0" ixz = "0"
+        iyy="${m*(x*x+z*z)/12}" iyz = "0"
+        izz="${m*(x*x+y*y)/12}"/>
+</xacro:macro>
+<xacro:macro name="cylinder_inertia" params="m r h">
+    <mass value="${m}" />
+    <inertia  ixx="${m*(3*r*r+h*h)/12}" ixy = "0" ixz = "0"
+        iyy="${m*(3*r*r+h*h)/12}" iyz = "0"
+        izz="${m*r*r/2}"/>
+</xacro:macro>
 <xacro:macro name="wheel_link" params="name pretty:=^|true wheelRadius:=^ wheelWidth:=^ wheelMass:=^">
     <link name="${name}">
         <inertial>
             <origin xyz="0 0 0" rpy="0 0 0" />
-            <mass value="${wheelMass}" />
-            <inertia
-                ixx="0.0059462"
-                ixy="0"
-                ixz="0"
-                iyy="0.0059468"
-                iyz="0"
-                izz="0.0072591" />
+            <xacro:cylinder_inertia m="${wheelMass}" r="${wheelRadius}" h="${wheelWidth}" />
         </inertial>
         <visual>
@@ -34,4 +39,8 @@
         </collision>
     </link>
+    <gazebo reference="${name}">
+        <mu1 value="1.0" />
+        <mu2 value="0.5" />
+    </gazebo>
 </xacro:macro>
 <xacro:macro name="wheel_joint" params="wheel x y z">

File: src/robot_description/models/master_ASM/urdf/master_ASM.urdf.xacro (robot description, xacro)
@@ -64,5 +64,5 @@
         <topic>joint_states</topic>
         </plugin>
-        <plugin
+        <!-- <plugin
         filename="ignition-gazebo-joint-controller-system"
         name="ignition::gazebo::systems::JointController">
@@ -87,4 +87,15 @@
         <joint_name>wheelBackRight_joint</joint_name>
         <initial_velocity>1.0</initial_velocity>
+        </plugin> -->
+        <plugin
+        filename="libignition-gazebo-diff-drive-system.so"
+        name="ignition::gazebo::systems::DiffDrive">
+          <left_joint>wheelFrontLeft_joint</left_joint>
+          <left_joint>wheelBackLeft_joint</left_joint>
+          <right_joint>wheelFrontRight_joint</right_joint>
+          <right_joint>wheelBackRight_joint</right_joint>
+          <wheel_separation>${chassisWidth + wheelWidth}</wheel_separation> <!-- ${chassisWidth + wheelWidth} 0.6177 -->
+          <wheel_radius>${wheelRadius}</wheel_radius> <!-- ${wheelRadius} 0.16 -->
+          <topic>cmd_vel</topic>
         </plugin>
     </gazebo>

File: src/robot_description/models/master_ASM/urdf/robot.urdf.xacro (robot description, xacro)
@@ -4,5 +4,5 @@
     <xacro:property name="chassisLength" value="1.13198"/>
     <xacro:property name="chassisWidth" value="0.5077"/>
-    <xacro:property name="chassisMass" value="55"/>
+    <xacro:property name="chassisMass" value="20"/>
     <xacro:property name="wheelWidth" value="0.11"/>
     <xacro:property name="wheelRadius" value="0.16"/>
@@ -12,5 +12,5 @@
     <!-- Distance from back of chassis to middle of back wheels 0.1534125 -->
     <!-- Distance from bottom of chassis to middle of wheels 0.0475 -->
-    <xacro:property name="wheelDeltaWidth" value="${(chassisWidth + wheelWidth)/2}" />
+    <xacro:property name="wheelDeltaWidth" value="${(chassisWidth + wheelWidth)/2}" /> <!-- not using messured distance because can calculate it-->
     <xacro:property name="wheelDeltaBack" value="-${chassisLength/2 - 0.1534125}" />
     <xacro:property name="wheelDeltaFront" value="${wheelDeltaBack + 0.873175}" />
@@ -24,13 +24,6 @@
     <link name="frame_link">
         <inertial>
-        <origin xyz="0 0 0" rpy="0 0 0" />
-        <mass value="${chassisMass}" />
-        <inertia
-            ixx="0.51975"
-            ixy="0"
-            ixz="0"
-            iyy="0.93889"
-            iyz="0"
-            izz="0.5273" />
+            <origin xyz="0 0 0" rpy="0 0 0" />
+            <xacro:box_inertia m="${chassisMass}" x="${chassisWidth}" y="${chassisLength}" z="${chassisHeight}" />
         </inertial>
         <visual>
