Commit message: camera that breaks shits

File: src/robot_description/models/master_ASM/urdf/master_ASM.urdf.xacro (robot description, xacro)
@@ -44,29 +44,36 @@
     </collision>
   </link>
-  <xacro:include filename="$(find zed_wrapper)/urdf/zed_macro.urdf.xacro" />
-  <xacro:zed_camera name="zed2i" model="zed2i">
-  </xacro:zed_camera>
+  <!-- <link name="camera_link">
+    <visual>
+      <origin
+        xyz="0 0 0.5"
+        rpy="1.57 0 1.57" />
+      <geometry>
+        <box size="0.1 0.1 0.1" />
+      </geometry>
+    </visual>
+  </link>
   <joint name="camera_joint" type="fixed">
-    <child link="base_link"/>
-    <parent link="zed2i_camera_link"/>
-    <origin xyz="-0.343 -0.009 -0.1254" rpy="0 -0.52359878 0" />
-  </joint>
-  <gazebo reference="zed2i_camera_link">
+      <parent link="base_link"/>
+      <child link="camera_link"/>
+      <origin xyz="0 0 0" rpy="0 0 0"/>
+  </joint> -->
+  <gazebo reference="base_link"> <!-- camera_link -->
     <sensor name="camera" type="camera">
-      <pose> 0 0 0 0 0 0 </pose>
-      <!-- <visualize>true</visualize> -->
-      <update_rate>30</update_rate>
+      <pose>0 0 0 0 0 0</pose>
       <camera>
-        <horizontal_fov>1.91986218</horizontal_fov>
+        <horizontal_fov>1.047</horizontal_fov>
         <image>
-          <format>R8G8B8</format>
-          <width>1280</width>
-          <height>720</height>
+          <width>320</width>
+          <height>240</height>
         </image>
         <clip>
-          <near>0.05</near>
-          <far>8.0</far>
+          <near>0.1</near>
+          <far>100</far>
         </clip>
       </camera>
+      <always_on>1</always_on>
+      <update_rate>15</update_rate>
+      <visualize>true</visualize>
       <topic>camera</topic>
     </sensor>
@@ -457,28 +464,28 @@
   </joint>
   <gazebo>
-    <plugin
-      filename="ignition-gazebo-joint-controller-system"
-      name="ignition::gazebo::systems::JointController">
-      <joint_name>wheel1_joint</joint_name>
-      <initial_velocity>0.0</initial_velocity>
-    </plugin>
-    <plugin
-      filename="ignition-gazebo-joint-controller-system"
-      name="ignition::gazebo::systems::JointController">
-      <joint_name>wheel2_joint</joint_name>
-      <initial_velocity>0.0</initial_velocity>
-    </plugin>
-    <plugin
-      filename="ignition-gazebo-joint-controller-system"
-      name="ignition::gazebo::systems::JointController">
-      <joint_name>wheel3_joint</joint_name>
-      <initial_velocity>0.0</initial_velocity>
-    </plugin>
-    <plugin
-      filename="ignition-gazebo-joint-controller-system"
-      name="ignition::gazebo::systems::JointController">
-      <joint_name>wheel4_joint</joint_name>
-      <initial_velocity>0.0</initial_velocity>
-    </plugin>
+  <plugin
+    filename="ignition-gazebo-joint-controller-system"
+    name="ignition::gazebo::systems::JointController">
+    <joint_name>wheel1_joint</joint_name>
+    <initial_velocity>0.0</initial_velocity>
+  </plugin>
+  <plugin
+    filename="ignition-gazebo-joint-controller-system"
+    name="ignition::gazebo::systems::JointController">
+    <joint_name>wheel2_joint</joint_name>
+    <initial_velocity>0.0</initial_velocity>
+  </plugin>
+  <plugin
+    filename="ignition-gazebo-joint-controller-system"
+    name="ignition::gazebo::systems::JointController">
+    <joint_name>wheel3_joint</joint_name>
+    <initial_velocity>0.0</initial_velocity>
+  </plugin>
+  <plugin
+    filename="ignition-gazebo-joint-controller-system"
+    name="ignition::gazebo::systems::JointController">
+    <joint_name>wheel4_joint</joint_name>
+    <initial_velocity>0.0</initial_velocity>
+  </plugin>
   </gazebo>
   <!-- model/Master_ASM/joint/{jointName}/cmd_vel -->
@@ -486,36 +493,36 @@
   <!-- model/Master_ASM/joint/{jointName}/0//cmd_pos -->
   <gazebo>
-    <plugin
-      filename="ignition-gazebo-joint-position-controller-system"
-      name="ignition::gazebo::systems::JointPositionController">
-      <joint_name>swerve1_joint</joint_name>
-      <use_velocity_commands>true</use_velocity_commands>
-      <cmd_max>15</cmd_max>
-      <cmd_min>-15</cmd_min>
-    </plugin>
-    <plugin
-      filename="ignition-gazebo-joint-position-controller-system"
-      name="ignition::gazebo::systems::JointPositionController">
-      <joint_name>swerve2_joint</joint_name>
-      <use_velocity_commands>true</use_velocity_commands>
-      <cmd_max>15</cmd_max>
-      <cmd_min>-15</cmd_min>
-    </plugin>
-    <plugin
-      filename="ignition-gazebo-joint-position-controller-system"
-      name="ignition::gazebo::systems::JointPositionController">
-      <joint_name>swerve3_joint</joint_name>
-      <use_velocity_commands>true</use_velocity_commands>
-      <cmd_max>15</cmd_max>
-      <cmd_min>-15</cmd_min>
-    </plugin>
-    <plugin
-      filename="ignition-gazebo-joint-position-controller-system"
-      name="ignition::gazebo::systems::JointPositionController">
-      <joint_name>swerve4_joint</joint_name>
-      <use_velocity_commands>true</use_velocity_commands>
-      <cmd_max>15</cmd_max>
-      <cmd_min>-15</cmd_min>
-    </plugin>
+  <plugin
+    filename="ignition-gazebo-joint-position-controller-system"
+    name="ignition::gazebo::systems::JointPositionController">
+    <joint_name>swerve1_joint</joint_name>
+    <use_velocity_commands>true</use_velocity_commands>
+    <cmd_max>15</cmd_max>
+    <cmd_min>-15</cmd_min>
+  </plugin>
+  <plugin
+    filename="ignition-gazebo-joint-position-controller-system"
+    name="ignition::gazebo::systems::JointPositionController">
+    <joint_name>swerve2_joint</joint_name>
+    <use_velocity_commands>true</use_velocity_commands>
+    <cmd_max>15</cmd_max>
+    <cmd_min>-15</cmd_min>
+  </plugin>
+  <plugin
+    filename="ignition-gazebo-joint-position-controller-system"
+    name="ignition::gazebo::systems::JointPositionController">
+    <joint_name>swerve3_joint</joint_name>
+    <use_velocity_commands>true</use_velocity_commands>
+    <cmd_max>15</cmd_max>
+    <cmd_min>-15</cmd_min>
+  </plugin>
+  <plugin
+    filename="ignition-gazebo-joint-position-controller-system"
+    name="ignition::gazebo::systems::JointPositionController">
+    <joint_name>swerve4_joint</joint_name>
+    <use_velocity_commands>true</use_velocity_commands>
+    <cmd_max>15</cmd_max>
+    <cmd_min>-15</cmd_min>
+  </plugin>
   </gazebo>
 </robot>

Commit message: like mostly works

File: src/robot_description/models/master_ASM/urdf/master_ASM.urdf.xacro (robot description, xacro)
@@ -59,5 +59,5 @@
       <origin xyz="0 0 0" rpy="0 0 0"/>
   </joint> -->
-  <gazebo reference="base_link"> <!-- camera_link -->
+  <!-- <gazebo reference="base_link"> camera_link
     <sensor name="camera" type="camera">
       <pose>0 0 0 0 0 0</pose>
@@ -78,5 +78,48 @@
       <topic>camera</topic>
     </sensor>
-  </gazebo>
+  </gazebo> -->
+  <joint name="camera_joint" type="fixed">
+        <parent link="base_link"/>
+        <child link="camera_link"/>
+        <origin xyz="0.305 0 0.08" rpy="0 0 0"/>
+    </joint>
+    <link name="camera_link">
+        <visual>
+            <geometry>
+                <box size="0.010 0.03 0.03"/>
+            </geometry>
+            <!-- <material name="red"/> -->
+        </visual>
+    </link>
+    <!-- <joint name="camera_optical_joint" type="fixed">
+        <parent link="camera_link"/>
+        <child link="camera_link_optical"/>
+        <origin xyz="0 0 0" rpy="1.57 0 1.57"/>
+    </joint>
+    <link name="camera_link_optical"></link> -->
+    <gazebo reference="camera_link">
+        <sensor name="camera" type="camera">
+            <pose> 0 0 0 0 0 0 </pose>
+            <!-- <visualize>true</visualize> -->
+            <update_rate>31</update_rate>
+            <camera>
+                <horizontal_fov>1.91986</horizontal_fov>
+                <vertical_fov>1.22173</vertical_fov>
+                <image>
+                    <format>R8G8B8</format>
+                    <width>1280</width>
+                    <height>720</height>
+                </image>
+                <clip>
+                    <near>0.05</near>
+                    <far>8.0</far>
+                </clip>
+            </camera>
+            <topic>camera</topic>
+            <!-- <plugin name="camera_controller" filename="libgazebo_ros_camera.so">
+                <frame_name>camera_link_optical</frame_name>
+            </plugin> -->
+        </sensor>
+    </gazebo>
   <link
     name="swerve1_Link">

Commit message: depth and camera box correct size

File: src/robot_description/models/master_ASM/urdf/master_ASM.urdf.xacro (robot description, xacro)
@@ -82,10 +82,10 @@
         <parent link="base_link"/>
         <child link="camera_link"/>
-        <origin xyz="0.305 0 0.08" rpy="0 0 0"/>
+        <origin xyz="0.35 0 0.05" rpy="0 0 0"/>
     </joint>
     <link name="camera_link">
         <visual>
             <geometry>
-                <box size="0.010 0.03 0.03"/>
+                <box size="0.03025 0.17525 0.04310"/>
             </geometry>
             <!-- <material name="red"/> -->
@@ -102,8 +102,7 @@
             <pose> 0 0 0 0 0 0 </pose>
             <!-- <visualize>true</visualize> -->
-            <update_rate>31</update_rate>
+            <update_rate>30</update_rate>
             <camera>
                 <horizontal_fov>1.91986</horizontal_fov>
-                <vertical_fov>1.22173</vertical_fov>
                 <image>
                     <format>R8G8B8</format>
@@ -117,7 +116,22 @@
             </camera>
             <topic>camera</topic>
-            <!-- <plugin name="camera_controller" filename="libgazebo_ros_camera.so">
-                <frame_name>camera_link_optical</frame_name>
-            </plugin> -->
+        </sensor>
+        <sensor name="depthcamera" type="depth">
+            <pose> 0 0 0 0 0 0 </pose>
+            <!-- <visualize>true</visualize> -->
+            <update_rate>30</update_rate>
+            <camera>
+                <horizontal_fov>1.91986</horizontal_fov>
+                <image>
+                    <format>R8G8B8</format>
+                    <width>1280</width>
+                    <height>720</height>
+                </image>
+                <clip>
+                    <near>0.05</near>
+                    <far>100.0</far>
+                </clip>
+            </camera>
+            <topic>depth</topic>
         </sensor>
     </gazebo>

Commit message: Sync with main branch

File: src/robot_description/models/master_ASM/urdf/master_ASM.urdf.xacro (robot description, xacro)
@@ -44,96 +44,50 @@
     </collision>
   </link>
-  <!-- <link name="camera_link">
-    <visual>
-      <origin
-        xyz="0 0 0.5"
-        rpy="1.57 0 1.57" />
-      <geometry>
-        <box size="0.1 0.1 0.1" />
-      </geometry>
-    </visual>
-  </link>
   <joint name="camera_joint" type="fixed">
       <parent link="base_link"/>
       <child link="camera_link"/>
-      <origin xyz="0 0 0" rpy="0 0 0"/>
-  </joint> -->
-  <!-- <gazebo reference="base_link"> camera_link
-    <sensor name="camera" type="camera">
-      <pose>0 0 0 0 0 0</pose>
-      <camera>
-        <horizontal_fov>1.047</horizontal_fov>
-        <image>
-          <width>320</width>
-          <height>240</height>
-        </image>
-        <clip>
-          <near>0.1</near>
-          <far>100</far>
-        </clip>
-      </camera>
-      <always_on>1</always_on>
-      <update_rate>15</update_rate>
-      <visualize>true</visualize>
-      <topic>camera</topic>
-    </sensor>
-  </gazebo> -->
-  <joint name="camera_joint" type="fixed">
-        <parent link="base_link"/>
-        <child link="camera_link"/>
-        <origin xyz="0.35 0 0.05" rpy="0 0 0"/>
-    </joint>
-    <link name="camera_link">
-        <visual>
-            <geometry>
-                <box size="0.03025 0.17525 0.04310"/>
-            </geometry>
-            <!-- <material name="red"/> -->
-        </visual>
-    </link>
-    <!-- <joint name="camera_optical_joint" type="fixed">
-        <parent link="camera_link"/>
-        <child link="camera_link_optical"/>
-        <origin xyz="0 0 0" rpy="1.57 0 1.57"/>
-    </joint>
-    <link name="camera_link_optical"></link> -->
-    <gazebo reference="camera_link">
-        <sensor name="camera" type="camera">
-            <pose> 0 0 0 0 0 0 </pose>
-            <!-- <visualize>true</visualize> -->
-            <update_rate>30</update_rate>
-            <camera>
-                <horizontal_fov>1.91986</horizontal_fov>
-                <image>
-                    <format>R8G8B8</format>
-                    <width>1280</width>
-                    <height>720</height>
-                </image>
-                <clip>
-                    <near>0.05</near>
-                    <far>8.0</far>
-                </clip>
-            </camera>
-            <topic>camera</topic>
-        </sensor>
-        <sensor name="depthcamera" type="depth">
-            <pose> 0 0 0 0 0 0 </pose>
-            <!-- <visualize>true</visualize> -->
-            <update_rate>30</update_rate>
-            <camera>
-                <horizontal_fov>1.91986</horizontal_fov>
-                <image>
-                    <format>R8G8B8</format>
-                    <width>1280</width>
-                    <height>720</height>
-                </image>
-                <clip>
-                    <near>0.05</near>
-                    <far>100.0</far>
-                </clip>
-            </camera>
-            <topic>depth</topic>
-        </sensor>
-    </gazebo>
+      <origin xyz="0.35 0 0.05" rpy="0 0 0"/>
+  </joint>
+  <link name="camera_link">
+    <visual>
+      <geometry>
+        <mesh filename="../meshes/zed2i.stl" />
+      </geometry>
+      <material name="zed2i_mat">
+        <color rgba="0.25 0.25 0.25 0.99"/>
+      </material>
+    </visual>
+    <collision>
+      <geometry>
+        <mesh filename="../meshes/zed2i.stl" />
+      </geometry>
+    </collision>
+  </link>
+  <!-- <joint name="camera_optical_joint" type="fixed">
+      <parent link="camera_link"/>
+      <child link="camera_link_optical"/>
+      <origin xyz="0 0 0" rpy="1.57 0 1.57"/>
+  </joint>
+  <link name="camera_link_optical"></link> -->
+  <gazebo reference="camera_link">
+      <sensor name="camera" type="camera">
+          <pose> 0 0 0 0 0 0 </pose>
+          <!-- <visualize>true</visualize> -->
+          <update_rate>30</update_rate>
+          <camera>
+              <horizontal_fov>1.91986</horizontal_fov>
+              <image>
+                  <format>R8G8B8</format>
+                  <width>1280</width>
+                  <height>720</height>
+              </image>
+              <clip>
+                  <near>0.05</near>
+                  <far>8.0</far>
+              </clip>
+          </camera>
+          <topic>camera</topic>
+      </sensor>
+  </gazebo>
   <link
     name="swerve1_Link">
