Commit message: Rework code so robot frame is base_link is the center of the robot instead of the zed (#221)
* depth camera

Removed depth topic stuff

Update container build process
Zed modules removed in support of local volume mount
gitignore updated to support custom mounts not being updated
Added cached layers for realsense to reduce buildtimes

switched from printf to echo and deleted \n from echo command

Deleted Extra Rocks from Gazebo

Merge the "URDF" branch into main (finally!) (#167)

* Update robot base frame and RViz configuration
Setup work to creat robot visualization

* Instantiated sweremodules

* Implemented the methods for power and angle

* Began changing tank drive code into swerve code in drive method

* minor cleanup

* Squashed commit of the following:

commit 01d3d55044bd4fbed79aa60882807ab722dd9f7f
Author: Anthony Brogni <anthonybrog@gmail.com>
Date:   Wed Oct 25 21:58:33 2023 -0500

    Simplify our code by adding all of the VESCs to the hashmap at the beginning

commit 709710e458619891ff8bb2666acf32d781476b39
Author: Anthony Brogni <anthonybrog@gmail.com>
Date:   Wed Oct 25 21:52:01 2023 -0500

    Added more TODOs

commit c0a9e65136265b8b0a28e7e08fbd508b362875b2
Author: Anthony Brogni <anthonybrog@gmail.com>
Date:   Wed Oct 25 21:45:39 2023 -0500

    Added TODOs

commit abc43a953e98f09255d290e3a8ddadc3f35aaa36
Author: Anthony Brogni <anthonybrog@gmail.com>
Date:   Wed Oct 25 21:43:09 2023 -0500

    minor cleanup

commit d87807716f8e3e88bbb4cfd4f3346ab10a192ab2
Author: Anthony Brogni <anthonybrog@gmail.com>
Date:   Wed Oct 25 01:46:32 2023 +0000

    switch to master of ros2socketcan_bridge

commit be8428cd46347b9cd319162d1bb62286ba1a0c3e
Author: umnrobotics <robotics@umn.edu>
Date:   Tue Oct 24 19:12:55 2023 -0500

    can

commit 1dd95159bf88c93fe7134e119ac2bc037197b733
Author: umnrobotics <robotics@umn.edu>
Date:   Tue Oct 24 19:02:10 2023 -0500

    floating point division

commit 341151ac295b430d209275b9fac0b3bfb7edc5db
Author: Anthony Brogni <anthonybrog@gmail.com>
Date:   Wed Oct 18 20:58:22 2023 -0500

    Delete .isaac_ros_common-config

commit b19663191ef392851531d651b8947eee68a9096b
Author: Anthony Brogni <anthonybrog@gmail.com>
Date:   Wed Oct 18 20:58:04 2023 -0500

    Removed these weird files

commit 11f8bb3c73ccdf74f7c2976310028a08c8fed76e
Merge: 8f67ce6 d49083f
Author: umnrobotics <robotics@umn.edu>
Date:   Wed Oct 18 19:36:45 2023 -0500

    Merge branch 'VESC-control-improvement' of github.com:GOFIRST-Robotics/Lunabotics-2024 into VESC-control-improvement

commit 8f67ce677da0013ec1b33fe8b7d6c6736b221e96
Author: umnrobotics <robotics@umn.edu>
Date:   Wed Oct 18 19:36:02 2023 -0500

    Set all defaults to 0

commit d49083f068521ee602b1304074f170ab14ba467a
Author: Derek <wderekgg@gmail.com>
Date:   Wed Oct 18 18:49:22 2023 -0500

    Value of Position is in degrees

commit edf339d69b343473f8035b9d6debcc35f0c5ac36
Author: Derek <wderekgg@gmail.com>
Date:   Wed Oct 18 18:37:49 2023 -0500

    Added Comments

commit c57985ad2a2e85606644dbdf6094ba252afdbca4
Merge: e0f9d20 a51c648
Author: Anthony Brogni <anthonybrog@gmail.com>
Date:   Wed Oct 18 11:29:28 2023 -0500

    Merge branch 'main' into VESC-control-improvement

commit e0f9d20effb19b5ad89ad95d97963cf6b3ac3de1
Merge: c03336d 5d0db07
Author: Anthony Brogni <anthonybrog@gmail.com>
Date:   Tue Oct 17 21:35:55 2023 -0500

    Merge branch 'main' into VESC-control-improvement

commit c03336d13e7db8389eaf5ea8a189408fd4e3dbd5
Merge: 376ad38 156950d
Author: Anthony Brogni <anthonybrog@gmail.com>
Date:   Sun Oct 15 17:49:16 2023 -0500

    Merge branch 'main' into VESC-control-improvement

commit 376ad3855895150d290fbf080d01c340cf4e7b6f
Author: Anthony Brogni <anthonybrog@gmail.com>
Date:   Sun Oct 15 17:49:10 2023 -0500

    minor cleanup

commit 17a06964580424f4d6d0a455cec4b41f390cea96
Merge: d3dfd7e 87189a8
Author: Anthony Brogni <anthonybrog@gmail.com>
Date:   Wed Oct 11 20:59:53 2023 -0500

    Merge branch 'main' into VESC-control-improvement

commit d3dfd7ef3563d40f9f3212f32df875b45bd23e14
Author: umnrobotics <robotics@umn.edu>
Date:   Wed Oct 11 19:34:22 2023 -0500

    Updated id names and commented out update

commit d4a16dcd618f21828c1397c05e84ec0801b20e43
Author: Adam Yaj <yaj00002@umn.edu>
Date:   Wed Oct 11 23:53:24 2023 +0000

    Added set position and set current code

    Co-authored-by: UMN Robotics <umnrobotics@users.noreply.github.com>
    Co-authored-by: sfisher9793 <sfisher9793@users.noreply.github.com>

commit 2e4570de483c147102c45d0b4ca8f0158b9182b0
Author: Adam Yaj <yaj00002@umn.edu>
Date:   Wed Oct 11 23:24:14 2023 +0000

    Updated CAN_callback to use Switch Statment

commit 5362e70b2294194e80f8718bba77cd6827f68cbb
Author: alex <whatshisname303@gmail.com>
Date:   Tue Oct 10 19:04:20 2023 -0500

    Update CAN_callback

* Update drivetrain_node.py

* Implemented inverse swerve drive equations

* Modified joystick inputs

* Fixed bugs

* Implemented optimal steering

* Revert "Implemented optimal steering"

This reverts commit 0f761afbac18adb9ccd457388fd212177ee0bdf7.

* Autoformatting Cleanup

* Revert "Squashed commit of the following:"

This reverts commit 01fa2c5d60a5fb5e625235f134a6a1d1986779f8.

* Update ros2socketcan_bridge

* Revert "Update ros2socketcan_bridge"

This reverts commit 8f0179eb39caba06ddf9c281f7c9f5eacf0446f9.

* Update main_control_node.py

* Update drivetrain_node.py

* Use set_state instead

* made a config file

* Update ros2socketcan_bridge

---------

Co-authored-by: akshatarinav <akshatarinav@gmail.com>
Co-authored-by: Shurderfer <aaron@kurlykris.com>
Co-authored-by: umnrobotics <robotics@umn.edu>
Co-authored-by: Jonathan Blixt <jmblixt3@gmail.com>

* motor_control_node Improvements (#96)

* Update CAN_callback

* Updated CAN_callback to use Switch Statment

* Added set position and set current code

Co-authored-by: UMN Robotics <umnrobotics@users.noreply.github.com>
Co-authored-by: sfisher9793 <sfisher9793@users.noreply.github.com>

* Updated id names and commented out update

* minor cleanup

* Added Comments

* Value of Position is in degrees

* Set all defaults to 0

* Removed these weird files

* Delete .isaac_ros_common-config

* floating point division

* can

* switch to master of ros2socketcan_bridge

* minor cleanup

* Added TODOs

* Added more TODOs

* Simplify our code by adding all of the VESCs to the hashmap at the beginning

* Revert "Simplify our code by adding all of the VESCs to the hashmap at the beginning"

This reverts commit 01d3d55044bd4fbed79aa60882807ab722dd9f7f.

* minor changes

* Update motor_control_node.cpp

* Added Basic Tachometer Feedback

* Added Structure For PID Position Control

* Revert "Added Structure For PID Position Control"

This reverts commit f84b982c5494c798d66ba503477bf3a5ebf066da.

* Revert "Added Basic Tachometer Feedback"

This reverts commit 2979c6d13f3b462f672ab2f4cc27f9834b4678cc.

* Update motor_control_node.cpp

* Update motor_control_node.cpp

* Added a config file for motor_control

* make use of std::optional instead of sentinal values

---------

Co-authored-by: alex <whatshisname303@gmail.com>
Co-authored-by: Adam Yaj <yaj00002@umn.edu>
Co-authored-by: UMN Robotics <umnrobotics@users.noreply.github.com>
Co-authored-by: sfisher9793 <sfisher9793@users.noreply.github.com>
Co-authored-by: umnrobotics <robotics@umn.edu>
Co-authored-by: Derek <wderekgg@gmail.com>

* Update zed ref

* Delete ros-bags directory

LFS is maxed out this fixes that issue

* Update zed_wrapper to use correct bag directory
lfs remove and updated directory

* fixed logging statements (#99)

* fixed logging in motor_control

* fixed python print statements

* std::optional bug fix

* Implemented Skimmer Height Adjustment (#100)

* Initial Commit

* remove incline methods

* remove Arduino code

* implemented SetHeight.srv, set height functions in conveyor_node

* cleanup

* finished refactoring our old conveyor idea (linear actuators) into the new idea (pulley system)

* Added more TODOs!

* Remove Arduino linear actuator controls from our repo

* Remove linear_actuator ROS parameters

* Created a new ROS param for manual height adjust

* Added publisher and height adjust methods

* Update MotorCommandGet.srv

* Create a publisher and timer for heigth adjust,
created method and service wrappers

* stop pulley,set pulley power+callbacks

* minor cleanup

* Squashed commit of the following:

commit 01d3d55044bd4fbed79aa60882807ab722dd9f7f
Author: Anthony Brogni <anthonybrog@gmail.com>
Date:   Wed Oct 25 21:58:33 2023 -0500

    Simplify our code by adding all of the VESCs to the hashmap at the beginning

commit 709710e458619891ff8bb2666acf32d781476b39
Author: Anthony Brogni <anthonybrog@gmail.com>
Date:   Wed Oct 25 21:52:01 2023 -0500

    Added more TODOs

commit c0a9e65136265b8b0a28e7e08fbd508b362875b2
Author: Anthony Brogni <anthonybrog@gmail.com>
Date:   Wed Oct 25 21:45:39 2023 -0500

    Added TODOs

commit abc43a953e98f09255d290e3a8ddadc3f35aaa36
Author: Anthony Brogni <anthonybrog@gmail.com>
Date:   Wed Oct 25 21:43:09 2023 -0500

    minor cleanup

commit d87807716f8e3e88bbb4cfd4f3346ab10a192ab2
Author: Anthony Brogni <anthonybrog@gmail.com>
Date:   Wed Oct 25 01:46:32 2023 +0000

    switch to master of ros2socketcan_bridge

commit be8428cd46347b9cd319162d1bb62286ba1a0c3e
Author: umnrobotics <robotics@umn.edu>
Date:   Tue Oct 24 19:12:55 2023 -0500

    can

commit 1dd95159bf88c93fe7134e119ac2bc037197b733
Author: umnrobotics <robotics@umn.edu>
Date:   Tue Oct 24 19:02:10 2023 -0500

    floating point division

commit 341151ac295b430d209275b9fac0b3bfb7edc5db
Author: Anthony Brogni <anthonybrog@gmail.com>
Date:   Wed Oct 18 20:58:22 2023 -0500

    Delete .isaac_ros_common-config

commit b19663191ef392851531d651b8947eee68a9096b
Author: Anthony Brogni <anthonybrog@gmail.com>
Date:   Wed Oct 18 20:58:04 2023 -0500

    Removed these weird files

commit 11f8bb3c73ccdf74f7c2976310028a08c8fed76e
Merge: 8f67ce6 d49083f
Author: umnrobotics <robotics@umn.edu>
Date:   Wed Oct 18 19:36:45 2023 -0500

    Merge branch 'VESC-control-improvement' of github.com:GOFIRST-Robotics/Lunabotics-2024 into VESC-control-improvement

commit 8f67ce677da0013ec1b33fe8b7d6c6736b221e96
Author: umnrobotics <robotics@umn.edu>
Date:   Wed Oct 18 19:36:02 2023 -0500

    Set all defaults to 0

commit d49083f068521ee602b1304074f170ab14ba467a
Author: Derek <wderekgg@gmail.com>
Date:   Wed Oct 18 18:49:22 2023 -0500

    Value of Position is in degrees

commit edf339d69b343473f8035b9d6debcc35f0c5ac36
Author: Derek <wderekgg@gmail.com>
Date:   Wed Oct 18 18:37:49 2023 -0500

    Added Comments

commit c57985ad2a2e85606644dbdf6094ba252afdbca4
Merge: e0f9d20 a51c648
Author: Anthony Brogni <anthonybrog@gmail.com>
Date:   Wed Oct 18 11:29:28 2023 -0500

    Merge branch 'main' into VESC-control-improvement

commit e0f9d20effb19b5ad89ad95d97963cf6b3ac3de1
Merge: c03336d 5d0db07
Author: Anthony Brogni <anthonybrog@gmail.com>
Date:   Tue Oct 17 21:35:55 2023 -0500

    Merge branch 'main' into VESC-control-improvement

commit c03336d13e7db8389eaf5ea8a189408fd4e3dbd5
Merge: 376ad38 156950d
Author: Anthony Brogni <anthonybrog@gmail.com>
Date:   Sun Oct 15 17:49:16 2023 -0500

    Merge branch 'main' into VESC-control-improvement

commit 376ad3855895150d290fbf080d01c340cf4e7b6f
Author: Anthony Brogni <anthonybrog@gmail.com>
Date:   Sun Oct 15 17:49:10 2023 -0500

    minor cleanup

commit 17a06964580424f4d6d0a455cec4b41f390cea96
Merge: d3dfd7e 87189a8
Author: Anthony Brogni <anthonybrog@gmail.com>
Date:   Wed Oct 11 20:59:53 2023 -0500

    Merge branch 'main' into VESC-control-improvement

commit d3dfd7ef3563d40f9f3212f32df875b45bd23e14
Author: umnrobotics <robotics@umn.edu>
Date:   Wed Oct 11 19:34:22 2023 -0500

    Updated id names and commented out update

commit d4a16dcd618f21828c1397c05e84ec0801b20e43
Author: Adam Yaj <yaj00002@umn.edu>
Date:   Wed Oct 11 23:53:24 2023 +0000

    Added set position and set current code

    Co-authored-by: UMN Robotics <umnrobotics@users.noreply.github.com>
    Co-authored-by: sfisher9793 <sfisher9793@users.noreply.github.com>

commit 2e4570de483c147102c45d0b4ca8f0158b9182b0
Author: Adam Yaj <yaj00002@umn.edu>
Date:   Wed Oct 11 23:24:14 2023 +0000

    Updated CAN_callback to use Switch Statment

commit 5362e70b2294194e80f8718bba77cd6827f68cbb
Author: alex <whatshisname303@gmail.com>
Date:   Tue Oct 10 19:04:20 2023 -0500

    Update CAN_callback

* Update conveyor_node.py

* change CAN IDs

* degree<->meter conversion for height adjust

* Update conveyor_node.py

* refactored "conveyor" into "skimmer"

* improvements (but still not finished)

* Revert "Squashed commit of the following:"

This reverts commit f67ccf5bdc095b9a604c1f1febc78621a487d80e.

* Update check_load.py

* Revert motor_control_node changes

* move launch file

* Removed the git lfs rosbags

* main_control_node improvements

* fixed call_async() to get the current position!

* package version updates

---------

Co-authored-by: RohanLShah123 <shah0711@umn.edu>
Co-authored-by: theduccom <145524869+theduccom@users.noreply.github.com>

---------

Co-authored-by: Jonathan Blixt <jmblixt3@gmail.com>
Co-authored-by: akshatarinav <akshatarinav@gmail.com>
Co-authored-by: Shurderfer <aaron@kurlykris.com>
Co-authored-by: umnrobotics <robotics@umn.edu>
Co-authored-by: alex <whatshisname303@gmail.com>
Co-authored-by: Adam Yaj <yaj00002@umn.edu>
Co-authored-by: UMN Robotics <umnrobotics@users.noreply.github.com>
Co-authored-by: sfisher9793 <sfisher9793@users.noreply.github.com>
Co-authored-by: Derek <wderekgg@gmail.com>
Co-authored-by: RohanLShah123 <shah0711@umn.edu>
Co-authored-by: theduccom <145524869+theduccom@users.noreply.github.com>

* Updated the size of our URDF

* Sync with the main branch (#157)

* Update README.md

* Deleted the "point_processing" package

* Delete testReadXML.py

* Auto format launch files and other minor improvements

* added zed mesh to gazebo urdf and adjusted the robot_desc file for rviz nvblox visualization

---------

Co-authored-by: Jonathan Blixt <jmblixt3@gmail.com>
Co-authored-by: akshatarinav <akshatarinav@gmail.com>
Co-authored-by: Shurderfer <aaron@kurlykris.com>
Co-authored-by: umnrobotics <robotics@umn.edu>
Co-authored-by: alex <whatshisname303@gmail.com>
Co-authored-by: Adam Yaj <yaj00002@umn.edu>
Co-authored-by: UMN Robotics <umnrobotics@users.noreply.github.com>
Co-authored-by: sfisher9793 <sfisher9793@users.noreply.github.com>
Co-authored-by: Derek <wderekgg@gmail.com>
Co-authored-by: RohanLShah123 <shah0711@umn.edu>
Co-authored-by: theduccom <145524869+theduccom@users.noreply.github.com>

update isaac ros common ref

updated urdf formatting

fixed urdf formatting

fixed more formatting

Update Isaac_ros_common ref
Added support for deepstream sdk

Changed Nav2 footprint from a circle to a rectangle (#186)

* hazzaaaah

* rectangle footprint

---------

Co-authored-by: Rohan Shah <shah0711@umn.edu>
Co-authored-by: umnrobotics <robotics@umn.edu>

Auto format the skimmer nodes

(DRAFT) Drivetrain Testing Improvements (NOT READY YET)I (#190)

* Initial commit

* fixed absolute encoder offset usage

* Testing Changes

* sus can ids

* No need to call self.set_angle(0)

* Revert "No need to call self.set_angle(0)"

This reverts commit 90f378959ce4465bcce9cf94fbe670ba974d7a03.

* Fixed default param values

* moved absolute encoder counts into a config file

* Made deadband a tunable paramater

* verified track width and wheel base

* changed max turn speeds

* remove comment

---------

Co-authored-by: umnrobotics <robotics@umn.edu>

Removed old scripts and made a new one

Fixed ZED TFs for both Gazebo & RVIZ (#195)

* auto format config files + change zed min depth

* ZED TF Changes for both gazebo & rviz

* made base_link same as gazebo

minor clean up

remove unused method

Fixed the absolute encoder code (#192)

* fix

* fixed back_right

* absolute encoders fix

* formatting

* final formatting

---------

Co-authored-by: umnrobotics <robotics@umn.edu>
Co-authored-by: Peter M <pwmarshall@gmail.com>

NASA KSC field added in Gazebo (#200)

* NASA field

* April tags finished

* Fix camera oops

* Final Clean up of name change

* what comments

Implemented crater detection in Nvblox (#188)

* Updated ref to point to our nvblox dev repo

* update submodule ref

* Swapping back to 3d render.

* Updating submodule reference. (change to nvblox_node.cpp)

* moving slice height to config file rather than hard coding

* Updating slice height config names + submodule reference

* Code to combine esdf layers in a python node. needs testing

* Rough outline for merging 2 costmaps. Needs better super positioning.

* Cleanup + pointcloud inversion. no merging yet though

* 'successfully' combining the pointclouds. poor performance though

* cleaning up aranges

* Some easy optimizations to reduce memory,
Untested

* updating gitignore

* the path planning avoids the hole. Cleanup and testing needed!

* Changed rviz view

* added basic sigmoid function

* adding images for visualization

* Im an idiot

* Working crater avoidance + gaussian blur + fixed combine pointcloud

* Major clean up

* deleting test files/ images and setting license

* Comments and more cleanup

* changed nvblox submodule branch

* update submodule ref

* Added combine_esdf to the nvblox launch file

* remove ssh from gitignore

* minor change

* update nvblox submodule ref (missing t)

* Fixing PR comments.

* Adding config file to launch

---------

Co-authored-by: Jonathan Blixt <jmblixt3@gmail.com>
Co-authored-by: alex berg <aaberg333@gmail.com>

Added an IMU sensor + RVIZ layout improvements

minor fixes

We now publish to the /odom topic

Getting close !!

Made an odom TF publisher

this line isn't a thing

minor improvements

launch file for current working state

nvblox works now !! (kind of)

Added the robot state publisher

Fix rosdep definitions for combine_esdf
Also update Dockerfile.umn to add these dependencies

Fixed the isaac_ros_launch setup.py & package.xml files

* minor cleanup

* FOV change back

* Inital work on combined launch file for sim and env

* finished fixing camera fov

* small fix

* update odom_tf_publisher frame id names

* fixed the odom -> zed2i_camera_link tf

* renamed  odom_tf_publisher to frame_renamer

* minor changes

* extend walls down

* Moved NASA mesh to the right folder

* Added TF topic to the NASA field

* Update topic names over bridge

* Initial working changes

* Add odom_publisher node

* Work on fixing gazebo with new tf trree

* Cleanup changes on this branch will be rebased

* Refactor to reduce code duplication across sim vs real robot

* Fix urdf during compile time so there isn't a duplicated file in our code section's

* Some fixups and revisions
Reverted some uneeded changes
Complete imu removal from gazebo
Remove an unused import

* Revert test of no tilt

* Remove dead code in nvblox node

---------

Co-authored-by: Isopod00 <anthonybrog@gmail.com>
Co-authored-by: Peter M <pwmarshall@gmail.com>
Co-authored-by: umnrobotics <robotics@umn.edu>

File: src/robot_description/models/master_ASM/urdf/master_ASM.urdf.xacro (robot description, xacro)
@@ -48,10 +48,29 @@
   </xacro:zed_camera>
   <joint name="camera_joint" type="fixed">
-    <child link="base_link"/>
-    <parent link="zed2i_camera_link"/>
-    <origin xyz="-0.343 -0.009 -0.1254" rpy="0 -0.52359878 0" />
+    <parent link="base_link"/>
+    <child link="zed2i_camera_link"/>
+    <origin xyz="0.343 -0.009 -0.1254" rpy="0 -0.52359878 0" />
   </joint>
   <gazebo reference="zed2i_camera_link">
     <sensor name="camera" type="camera">
+      <!-- <visualize>true</visualize> -->
+      <always_on>true</always_on>
+      <update_rate>30</update_rate>
+      <camera>
+        <horizontal_fov>1.91986218</horizontal_fov>
+        <image>
+          <format>R8G8B8</format>
+          <width>1280</width>
+          <height>720</height>
+        </image>
+        <clip>
+          <near>0.3</near>
+          <far>5.0</far>
+        </clip>
+      </camera>
+      <topic>/color/image</topic>
+      <info_topic>/color/camera_info</info_topic>
+    </sensor>
+    <sensor name="depthcamera" type="depth">
       <!-- <visualize>true</visualize> -->
       <always_on>true</always_on>
@@ -69,13 +88,6 @@
         </clip>
       </camera>
-      <topic>camera</topic>
-    </sensor>
-    <sensor name="imu_sensor" type="imu">
-      <always_on>1</always_on>
-      <update_rate>1</update_rate>
-      <visualize>true</visualize>
-      <topic>imu</topic>
-      <plugin filename="libignition-gazebo-imu-system.so" name="ignition::gazebo::systems::Imu">
-      </plugin>
+      <topic>/depth/image</topic>
+      <info_topic>/depth/camera_info</info_topic>
     </sensor>
   </gazebo>

Commit message: fixed my zed tf setup

File: src/robot_description/models/master_ASM/urdf/master_ASM.urdf.xacro (robot description, xacro)
@@ -45,8 +45,8 @@
   </link>
   <!-- Connect the base_link to the new link with only a translation -->
-  <joint name="translation_end_to_base" type="fixed">
+  <joint name="base_to_translation_end" type="fixed">
     <parent link="base_link"/>
     <child link="translation_end_link"/>
-    <origin xyz="0.343 -0.009 0.1254" rpy="0 0 0"/>
+    <origin xyz="0.343 -0.009 -0.1254" rpy="0 0 0"/>
   </joint>
   <!-- Add a new link at the end of the translation vector -->
@@ -62,8 +62,8 @@
   <xacro:zed_camera name="zed2i" model="zed2i">
   </xacro:zed_camera>
-  <joint name="camera_to_translation_end" type="fixed">
+  <joint name="translation_end_to_camera" type="fixed">
     <parent link="translation_end_link"/>
     <child link="zed2i_camera_link"/>
-    <origin xyz="0 0 0" rpy="0 -0.52359878 0"/>
+    <origin xyz="0 0 0" rpy="0 0.52359878 0"/>
   </joint>
   <gazebo reference="zed2i_camera_link">
