Commit message: Make zed2i_camera_link base_link

File: src/robot_description/models/master_ASM/urdf/master_ASM.urdf.xacro (robot description, xacro)
@@ -6,5 +6,5 @@
 <robot name="Master_ASM" xmlns:xacro="http://www.ros.org/wiki/xacro">
   <link
-    name="base_link">
+    name="frame_link">
     <inertial>
       <origin
@@ -27,5 +27,5 @@
       <geometry>
         <mesh
-          filename="package://robot_description/models/master_ASM/meshes/base_link.STL" />
+          filename="package://robot_description/models/master_ASM/meshes/frame_link.STL" />
       </geometry>
       <material
@@ -44,9 +44,9 @@
     </collision>
   </link>
-  <!-- Connect the base_link to the new link with only a translation -->
+  <!-- Connect the frame_link to the new link with only a translation -->
   <joint name="base_to_translation_end" type="fixed">
-    <parent link="base_link"/>
-    <child link="translation_end_link"/>
-    <origin xyz="0.343 -0.009 -0.1254" rpy="0 0 0"/>
+    <child link="frame_link"/>
+    <parent link="translation_end_link"/>
+    <origin xyz="-0.343 0.009 0.1254" rpy="0 0 0"/>
   </joint>
   <!-- Add a new link at the end of the translation vector -->
@@ -63,7 +63,7 @@
   </xacro:zed_camera>
   <joint name="translation_end_to_camera" type="fixed">
-    <parent link="translation_end_link"/>
-    <child link="zed2i_camera_link"/>
-    <origin xyz="0 0 0" rpy="0 0.52359878 0"/>
+    <child link="translation_end_link"/>
+    <parent link="zed2i_camera_link"/>
+    <origin xyz="-0 0 0" rpy="0 -0.52359878 0"/>
   </joint>
   <gazebo reference="zed2i_camera_link">
@@ -146,5 +146,5 @@
       rpy="1.5708 0 0" />
     <parent
-      link="base_link" />
+      link="frame_link" />
     <child
       link="swerve1_Link" />
@@ -242,5 +242,5 @@
       rpy="1.5708 0 3.1416" />
     <parent
-      link="base_link" />
+      link="frame_link" />
     <child
       link="swerve2_Link" />
@@ -340,5 +340,5 @@
       rpy="1.5708 0 3.1416" />
     <parent
-      link="base_link" />
+      link="frame_link" />
     <child
       link="swerve3_Link" />
@@ -435,5 +435,5 @@
       rpy="1.5708 0 0" />
     <parent
-      link="base_link" />
+      link="frame_link" />
     <child
       link="swerve4_Link" />

Commit message: Drivetrain Testing Fixes

File: src/robot_description/models/master_ASM/urdf/master_ASM.urdf.xacro (robot description, xacro)
@@ -48,5 +48,5 @@
     <parent link="translation_end_link"/>
     <child link="frame_link"/>
-    <origin xyz="-0.343 0.009 0.1254" rpy="0 0 0"/>
+    <origin xyz="-0.5 0 0.375" rpy="0 0 -1.57"/>
   </joint>
   <!-- Add a new link at the end of the translation vector -->
@@ -58,5 +58,5 @@
     </inertial>
   </link>
-  <!-- Connect the new link to the camera_link with only a rotation -->
+  <!-- Connect the translation_end_link to the zed2i_camera_link with only a rotation -->
   <xacro:include filename="$(find zed_wrapper)/urdf/zed_macro.urdf.xacro" />
   <xacro:zed_camera name="zed2i" model="zed2i" enable_gnss="false">
@@ -67,5 +67,5 @@
     <parent link="zed2i_camera_link"/>
     <child link="translation_end_link"/>
-    <origin xyz="0 0 0" rpy="0 -0.44 0"/>
+    <origin xyz="0 0 0" rpy="0 0 0"/>
   </joint>
   <gazebo reference="zed2i_camera_link">
@@ -143,5 +143,5 @@
   <joint
     name="swerve1_joint"
-    type="fixed"> <!-- fixed -->
+    type="fixed">
     <origin
       xyz="-0.34701 0.55026 -0.59563"
@@ -239,5 +239,5 @@
   <joint
     name="swerve2_joint"
-    type="fixed"> <!-- fixed -->
+    type="fixed">
     <origin
       xyz="0.34701 -0.55026 -0.59563"
@@ -526,40 +526,3 @@
     </plugin>
   </gazebo>
-  <!-- model/Master_ASM/joint/{jointName}/cmd_vel -->
-  <!--  ignition::msgs::Double, topic name and type for plugins -->
-  <!-- model/Master_ASM/joint/{jointName}/0//cmd_pos -->
-  <gazebo>
-    <plugin
-      filename="ignition-gazebo-joint-position-controller-system"
-      name="ignition::gazebo::systems::JointPositionController">
-      <joint_name>swerve1_joint</joint_name>
-      <use_velocity_commands>true</use_velocity_commands>
-      <cmd_max>15</cmd_max>
-      <cmd_min>-15</cmd_min>
-    </plugin>
-    <plugin
-      filename="ignition-gazebo-joint-position-controller-system"
-      name="ignition::gazebo::systems::JointPositionController">
-      <joint_name>swerve2_joint</joint_name>
-      <use_velocity_commands>true</use_velocity_commands>
-      <cmd_max>15</cmd_max>
-      <cmd_min>-15</cmd_min>
-    </plugin>
-    <plugin
-      filename="ignition-gazebo-joint-position-controller-system"
-      name="ignition::gazebo::systems::JointPositionController">
-      <joint_name>swerve3_joint</joint_name>
-      <use_velocity_commands>true</use_velocity_commands>
-      <cmd_max>15</cmd_max>
-      <cmd_min>-15</cmd_min>
-    </plugin>
-    <plugin
-      filename="ignition-gazebo-joint-position-controller-system"
-      name="ignition::gazebo::systems::JointPositionController">
-      <joint_name>swerve4_joint</joint_name>
-      <use_velocity_commands>true</use_velocity_commands>
-      <cmd_max>15</cmd_max>
-      <cmd_min>-15</cmd_min>
-    </plugin>
-  </gazebo>
 </robot>

Commit message: Initial commit of ZED urdf changes and switched to gen_2 pose tracking

File: src/robot_description/models/master_ASM/urdf/master_ASM.urdf.xacro (robot description, xacro)
@@ -5,4 +5,12 @@
      For more information, please see http://wiki.ros.org/sw_urdf_exporter -->
 <robot name="Master_ASM" xmlns:xacro="http://www.ros.org/wiki/xacro">
+  <link name="root_link">
+    <origin xyz="0 0 0" rpy="0 0 0" />
+  </link>
+  <joint name="root_to_frame_joint" type="fixed">
+    <parent link="root_link" />
+    <child link="frame_link" />
+    <origin xyz="0 0 0" rpy="0 0 -1.5708" />
+  </joint>
   <link
     name="frame_link">
@@ -44,19 +52,6 @@
     </collision>
   </link>
-  <!-- Connect the frame_link to the new link with only a translation -->
-  <joint name="base_to_translation_end" type="fixed">
-    <parent link="translation_end_link"/>
-    <child link="frame_link"/>
-    <origin xyz="-0.5 0 0.375" rpy="0 0 -1.57"/>
-  </joint>
-  <!-- Add a new link at the end of the translation vector -->
-  <link name="translation_end_link">
-    <inertial>
-      <origin xyz="0 0 0" rpy="0 0 0"/>
-      <mass value="0.001"/>
-      <inertia ixx="0.0001" ixy="0" ixz="0" iyy="0.0001" iyz="0" izz="0.0001"/>
-    </inertial>
-  </link>
-  <!-- Connect the translation_end_link to the zed2i_camera_link with only a rotation -->
+  <!-- ZED 2i Camera -->
+  <xacro:arg name="use_zed_localization" default="true" />
   <xacro:include filename="$(find zed_wrapper)/urdf/zed_macro.urdf.xacro" />
   <xacro:zed_camera name="zed2i" model="zed2i" enable_gnss="false">
@@ -64,9 +59,21 @@
     <gnss_origin></gnss_origin>
   </xacro:zed_camera>
-  <joint name="translation_end_to_camera" type="fixed">
-    <parent link="zed2i_camera_link"/>
-    <child link="translation_end_link"/>
-    <origin xyz="0 0 0" rpy="0 0 0"/>
-  </joint>
+  <!-- Add a joint to connect the ZED 2i Camera model to the robot -->
+  <xacro:if value="$(arg use_zed_localization)">
+    <!-- ZED Localization -> The reference link is 'zed2i_camera_link' and 'root_link' is a child -->
+    <joint name="zed2i_joint" type="fixed">
+      <parent link="zed2i_camera_link"/>
+      <child link="root_link"/>
+      <origin xyz="-0.5 0 0.375" rpy="0 0 0"/>
+    </joint>
+  </xacro:if>
+  <xacro:unless value="$(arg use_zed_localization)">
+    <!-- NO ZED Localization -> 'zed2i_camera_link' is a child of 'root_link' -->
+    <joint name="zed2i_joint" type="fixed">
+      <parent link="root_link"/>
+      <child link="zed2i_camera_link"/>
+      <origin xyz="0.5 0 -0.375" rpy="0 0 0"/>
+    </joint>
+  </xacro:unless>
   <gazebo reference="zed2i_camera_link">
     <sensor name="camera" type="camera">

Commit message: Renamed "root_link" to "base_link" to match conventions

File: src/robot_description/models/master_ASM/urdf/master_ASM.urdf.xacro (robot description, xacro)
@@ -5,9 +5,9 @@
      For more information, please see http://wiki.ros.org/sw_urdf_exporter -->
 <robot name="Master_ASM" xmlns:xacro="http://www.ros.org/wiki/xacro">
-  <link name="root_link">
+  <link name="base_link">
     <origin xyz="0 0 0" rpy="0 0 0" />
   </link>
-  <joint name="root_to_frame_joint" type="fixed">
-    <parent link="root_link" />
+  <joint name="base_to_frame_joint" type="fixed">
+    <parent link="base_link" />
     <child link="frame_link" />
     <origin xyz="0 0 0" rpy="0 0 -1.5708" />
@@ -61,15 +61,15 @@
   <!-- Add a joint to connect the ZED 2i Camera model to the robot -->
   <xacro:if value="$(arg use_zed_localization)">
-    <!-- ZED Localization -> The reference link is 'zed2i_camera_link' and 'root_link' is a child -->
+    <!-- ZED Localization -> The reference link is 'zed2i_camera_link' and 'base_link' is a child -->
     <joint name="zed2i_joint" type="fixed">
       <parent link="zed2i_camera_link"/>
-      <child link="root_link"/>
+      <child link="base_link"/>
       <origin xyz="-0.5 0 0.375" rpy="0 0 0"/>
     </joint>
   </xacro:if>
   <xacro:unless value="$(arg use_zed_localization)">
-    <!-- NO ZED Localization -> 'zed2i_camera_link' is a child of 'root_link' -->
+    <!-- NO ZED Localization -> 'zed2i_camera_link' is a child of 'base_link' -->
     <joint name="zed2i_joint" type="fixed">
-      <parent link="root_link"/>
+      <parent link="base_link"/>
       <child link="zed2i_camera_link"/>
       <origin xyz="0.5 0 -0.375" rpy="0 0 0"/>

Commit message: Initial commit

File: src/robot_description/models/master_ASM/urdf/master_ASM.urdf.xacro (robot description, xacro)
@@ -1,58 +1,128 @@
 <?xml version="1.0" encoding="utf-8"?>
-<!-- This URDF was automatically created by SolidWorks to URDF Exporter! Originally created by
-Stephen Brawner (brawner@gmail.com)
-     Commit Version: 1.6.0-4-g7f85cfe  Build Version: 1.6.7995.38578
-     For more information, please see http://wiki.ros.org/sw_urdf_exporter -->
 <robot name="Master_ASM" xmlns:xacro="http://www.ros.org/wiki/xacro">
+  <xacro:property name="PI" value="3.1415926535897931"/>
+  <xacro:property name="chassisHeight" value="0.1"/>
+  <xacro:property name="chassisLength" value="0.8"/>
+  <xacro:property name="chassisWidth" value="0.5"/>
+  <xacro:property name="chassisMass" value="50"/>
+  <xacro:property name="wheelWidth" value="0.05"/>
+  <xacro:property name="wheelRadius" value="0.2"/>
+  <xacro:property name="wheelMass" value="5"/>
+  <xacro:macro name="box_inertia" params="m x y z">
+    <inertia  ixx="${m*(y*y+z*z)/12}" ixy = "0" ixz = "0"
+      iyy="${m*(x*x+z*z)/12}" iyz = "0"
+      izz="${m*(x*x+z*z)/12}"/>
+  </xacro:macro>
+  <xacro:macro name="cylinder_inertia" params="m r h">
+    <inertia  ixx="${m*(3*r*r+h*h)/12}" ixy = "0" ixz = "0"
+      iyy="${m*(3*r*r+h*h)/12}" iyz = "0"
+      izz="${m*r*r/2}"/>
+  </xacro:macro>
+  <material name="silver">
+    <color rgba="0.700 0.700 0.700 1.000"/>
+  </material>
   <link name="base_link">
-    <origin xyz="0 0 0" rpy="0 0 0" />
-  </link>
-  <joint name="base_to_frame_joint" type="fixed">
-    <parent link="base_link" />
-    <child link="frame_link" />
-    <origin xyz="0 0 0" rpy="0 0 -1.5708" />
-  </joint>
-  <link
-    name="frame_link">
-    <inertial>
-      <origin
-        xyz="0.0012829 -0.31468 -0.0059364"
-        rpy="0 0 0" />
-      <mass
-        value="38.039" />
-      <inertia
-        ixx="0.51975"
-        ixy="0.00069908"
-        ixz="2.9544E-06"
-        iyy="0.93889"
-        iyz="-3.8081E-06"
-        izz="0.5273" />
-    </inertial>
-    <visual>
-      <origin
-        xyz="0 0 0"
-        rpy="0 0 0" />
-      <geometry>
-        <mesh
-          filename="package://robot_description/models/master_ASM/meshes/frame_link.STL" />
-      </geometry>
-      <material
-        name="">
-        <color
-          rgba="0.79216 0.81961 0.93333 1" />
-      </material>
-    </visual>
-    <collision>
-      <origin
-        xyz="0 0 -0.2"
-        rpy="0 0 0" />
-      <geometry>
-        <box size="0.7317 1.4254 0.6435" />
+    <inertial>
+      <origin rpy="0 0 0" xyz="0 0.0 0.08835894305363262"/>
+      <mass value="${chassisMass}"/>
+      <xacro:box_inertia m="${chassisMass}" x="${chassisLength}" y="${chassisWidth}" z="${chassisHeight}"/>
+    </inertial>
+    <visual>
+      <origin rpy="0 0 0" xyz="0 0 0"/>
+      <geometry>
+        <mesh filename="package://robot_description/models/master_ASM/meshes/base_link.stl" scale="0.001 0.001 0.001"/>
+      </geometry>
+      <material name="silver"/>
+    </visual>
+    <collision>
+      <origin rpy="0 0 0" xyz="0 0 0"/>
+      <geometry>
+        <mesh filename="package://robot_description/models/master_ASM/meshes/base_link.stl" scale="0.001 0.001 0.001"/>
+      </geometry>
+    </collision>
+  </link>
+  <link name="right_front">
+    <inertial>
+      <origin rpy="0 0 0" xyz="-4.3576253716537394e-14 -0.022224999999999995 -2.736260904245835e-07"/>
+      <mass value="${wheelMass}"/>
+      <xacro:cylinder_inertia m="${wheelMass}" r="${wheelRadius}" h="${wheelWidth}"/>
+    </inertial>
+    <visual>
+      <origin rpy="0 0 0" xyz="-0.254 0.254 -0.101276"/>
+      <geometry>
+        <mesh filename="package://robot_description/models/master_ASM/meshes/right_front.stl" scale="0.001 0.001 0.001"/>
+      </geometry>
+      <material name="silver"/>
+    </visual>
+    <collision>
+      <origin rpy="0 0 0" xyz="-0.254 0.254 -0.101276"/>
+      <geometry>
+        <mesh filename="package://robot_description/models/master_ASM/meshes/right_front.stl" scale="0.001 0.001 0.001"/>
+      </geometry>
+    </collision>
+  </link>
+  <link name="left_front">
+    <inertial>
+      <origin rpy="0 0 0" xyz="-4.3576253716537394e-14 0.02222499999999994 -2.736260904245835e-07"/>
+      <mass value="${wheelMass}"/>
+      <xacro:cylinder_inertia m="${wheelMass}" r="${wheelRadius}" h="${wheelWidth}"/>
+    </inertial>
+    <visual>
+      <origin rpy="0 0 0" xyz="-0.254 -0.254 -0.101276"/>
+      <geometry>
+        <mesh filename="package://robot_description/models/master_ASM/meshes/left_front.stl" scale="0.001 0.001 0.001"/>
+      </geometry>
+      <material name="silver"/>
+    </visual>
+    <collision>
+      <origin rpy="0 0 0" xyz="-0.254 -0.254 -0.101276"/>
+      <geometry>
+        <mesh filename="package://robot_description/models/master_ASM/meshes/left_front.stl" scale="0.001 0.001 0.001"/>
+      </geometry>
+    </collision>
+  </link>
+  <link name="left_back">
+    <inertial>
+      <origin rpy="0 0 0" xyz="-4.346523141407488e-14 0.02222499999999994 -2.7362609036907237e-07"/>
+      <mass value="${wheelMass}"/>
+      <xacro:cylinder_inertia m="${wheelMass}" r="${wheelRadius}" h="${wheelWidth}"/>
+    </inertial>
+    <visual>
+      <origin rpy="0 0 0" xyz="0.254 -0.254 -0.101276"/>
+      <geometry>
+        <mesh filename="package://robot_description/models/master_ASM/meshes/left_back.stl" scale="0.001 0.001 0.001"/>
+      </geometry>
+      <material name="silver"/>
+    </visual>
+    <collision>
+      <origin rpy="0 0 0" xyz="0.254 -0.254 -0.101276"/>
+      <geometry>
+        <mesh filename="package://robot_description/models/master_ASM/meshes/left_back.stl" scale="0.001 0.001 0.001"/>
+      </geometry>
+    </collision>
+  </link>
+  <link name="right_back">
+    <inertial>
+      <origin rpy="0 0 0" xyz="-4.3520742565306136e-14 -0.022224999999999995 -2.736260904245835e-07"/>
+      <mass value="${wheelMass}"/>
+      <xacro:cylinder_inertia m="${wheelMass}" r="${wheelRadius}" h="${wheelWidth}"/>
+    </inertial>
+    <visual>
+      <origin rpy="0 0 0" xyz="0.254 0.254 -0.101276"/>
+      <geometry>
+        <mesh filename="package://robot_description/models/master_ASM/meshes/right_back.stl" scale="0.001 0.001 0.001"/>
+      </geometry>
+      <material name="silver"/>
+    </visual>
+    <collision>
+      <origin rpy="0 0 0" xyz="0.254 0.254 -0.101276"/>
+      <geometry>
+        <mesh filename="package://robot_description/models/master_ASM/meshes/right_back.stl" scale="0.001 0.001 0.001"/>
       </geometry>
     </collision>
   </link>
   <!-- ZED 2i Camera -->
-  <xacro:arg name="use_zed_localization" default="true" />
-  <xacro:include filename="$(find zed_wrapper)/urdf/zed_macro.urdf.xacro" />
+  <xacro:arg name="use_zed_localization" default="true"/>
+  <xacro:include filename="$(find zed_wrapper)/urdf/zed_macro.urdf.xacro"/>
   <xacro:zed_camera name="zed2i" model="zed2i" enable_gnss="false">
     <!-- This block is required even if enable_gnss="false" for some reason, but you can leave it empty -->
@@ -118,387 +188,27 @@
     </sensor>
   </gazebo>
-  <link
-    name="swerve1_Link">
-    <inertial>
-      <origin
-        xyz="0.072878 0.028694 7.0574E-06"
-        rpy="0 0 0" />
-      <mass
-        value="2.5211" />
-      <inertia
-        ixx="0.008233"
-        ixy="5.8978E-05"
-        ixz="5.7912E-08"
-        iyy="0.006818"
-        iyz="1.2459E-07"
-        izz="0.0069443" />
-    </inertial>
-    <visual>
-      <origin
-        xyz="0 0 0"
-        rpy="0 0 0" />
-      <geometry>
-        <box size="0.1 0.2 0.1" />
-      </geometry>
-      <material
-        name="">
-        <color
-          rgba="0.75294 0.75294 0.75294 1" />
-      </material>
-    </visual>
-  </link>
-  <joint
-    name="swerve1_joint"
-    type="fixed">
-    <origin
-      xyz="-0.34701 0.55026 -0.59563"
-      rpy="1.5708 0 0" />
-    <parent
-      link="frame_link" />
-    <child
-      link="swerve1_Link" />
-    <axis
-      xyz="0 1 0" />
-    <!-- <limit lower="6.28" upper="6.28" effort="30" velocity="1.0" /> -->
-  </joint>
-  <link
-    name="wheel1_Link">
-    <inertial>
-      <origin
-        xyz="2.9097E-09 -0.115 -0.00055956"
-        rpy="0 0 0" />
-      <mass
-        value="1.1372" />
-      <inertia
-        ixx="0.0059462"
-        ixy="1.6529E-09"
-        ixz="-6.3363E-10"
-        iyy="0.0059468"
-        iyz="6.9163E-09"
-        izz="0.0072591" />
-    </inertial>
-    <visual>
-      <origin
-        xyz="0 0.115 0"
-        rpy="0 0 0" />
-      <geometry>
-        <mesh
-          filename="package://robot_description/models/master_ASM/meshes/wheel_Link.STL" />
-      </geometry>
-      <material
-        name="">
-        <color
-          rgba="0.79216 0.81961 0.93333 1" />
-      </material>
-    </visual>
-    <collision>
-      <origin
-        xyz="0 0 0"
-        rpy="0 0 0" />
-      <geometry>
-        <cylinder radius="0.115" length="0.2" />
-      </geometry>
-    </collision>
-  </link>
-  <joint
-    name="wheel1_joint"
-    type="continuous">
-    <origin
-      xyz="0 0 0"
-      rpy="1.5708 0.34561 1.5708" />
-    <parent
-      link="swerve1_Link" />
-    <child
-      link="wheel1_Link" />
-    <axis
-      xyz="0 0 -1" />
-  </joint>
-  <link
-    name="swerve2_Link">
-    <inertial>
-      <origin
-        xyz="0.072878 0.028694 7.0574E-06"
-        rpy="0 0 0" />
-      <mass
-        value="2.5211" />
-      <inertia
-        ixx="0.008233"
-        ixy="5.8978E-05"
-        ixz="5.7912E-08"
-        iyy="0.006818"
-        iyz="1.2459E-07"
-        izz="0.0069443" />
-    </inertial>
-    <visual>
-      <origin
-        xyz="0 0 0"
-        rpy="0 0 0" />
-      <geometry>
-        <box size="0.1 0.2 0.1" />
-      </geometry>
-      <material
-        name="">
-        <color
-          rgba="0.75294 0.75294 0.75294 1" />
-      </material>
-    </visual>
-  </link>
-  <joint
-    name="swerve2_joint"
-    type="fixed">
-    <origin
-      xyz="0.34701 -0.55026 -0.59563"
-      rpy="1.5708 0 3.1416" />
-    <parent
-      link="frame_link" />
-    <child
-      link="swerve2_Link" />
-    <axis
-      xyz="0 1 0" />
-    <!-- <limit lower="6.28" upper="6.28" effort="30" velocity="1.0" /> -->
-  </joint>
-  <link
-    name="wheel2_Link">
-    <inertial>
-      <origin
-        xyz="2.9097E-09 -0.115 -0.00055956"
-        rpy="0 0 0" />
-      <mass
-        value="1.1372" />
-      <inertia
-        ixx="0.0059462"
-        ixy="1.6529E-09"
-        ixz="-6.3363E-10"
-        iyy="0.0059468"
-        iyz="6.9163E-09"
-        izz="0.0072591" />
-    </inertial>
-    <visual>
-      <origin
-        xyz="0 0.115 0"
-        rpy="0 0 0" />
-      <geometry>
-        <mesh
-          filename="package://robot_description/models/master_ASM/meshes/wheel_Link.STL" />
-      </geometry>
-      <material
-        name="">
-        <color
-          rgba="0.79216 0.81961 0.93333 1" />
-      </material>
-    </visual>
-    <collision>
-      <origin
-        xyz="0 0 0"
-        rpy="0 0 0" />
-      <geometry>
-        <!-- <mesh
-          filename="package://Master_ASM/meshes/wheel2_Link.STL" /> -->
-        <cylinder radius="0.115" length="0.2" />
-      </geometry>
-    </collision>
-  </link>
-  <joint
-    name="wheel2_joint"
-    type="continuous">
-    <origin
-      xyz="0 0 0"
-      rpy="1.5708 0.34561 1.5708" />
-    <parent
-      link="swerve2_Link" />
-    <child
-      link="wheel2_Link" />
-    <axis
-      xyz="0 0 1" />
-  </joint>
-  <link
-    name="swerve3_Link">
-    <inertial>
-      <origin
-        xyz="0.072878 0.028694 7.0574E-06"
-        rpy="0 0 0" />
-      <mass
-        value="2.5211" />
-      <inertia
-        ixx="0.008233"
-        ixy="5.8978E-05"
-        ixz="5.7912E-08"
-        iyy="0.006818"
-        iyz="1.2459E-07"
-        izz="0.0069443" />
-    </inertial>
-    <visual>
-      <origin
-        xyz="0 0 0"
-        rpy="0 0 0" />
-      <geometry>
-        <box size="0.1 0.2 0.1" />
-      </geometry>
-      <material
-        name="">
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