Commit message: urdf fixes

File: src/robot_description/models/master_ASM/urdf/master_ASM.urdf.xacro (robot description, xacro)
@@ -23,6 +23,14 @@
   </material>
   <link name="base_link">
-    <inertial>
-      <origin rpy="0 0 0" xyz="0 0.0 0.08835894305363262"/>
+    <origin xyz="0 0 0" rpy="0 0 0"/>
+  </link>
+  <joint name="base_to_frame_joint" type="fixed">
+    <parent link="base_link"/>
+    <child link="frame_link"/>
+    <origin xyz="0 0 0" rpy="0 0 0"/>
+  </joint>
+  <link name="frame_link">
+    <inertial>
+      <origin xyz="0 0 0" rpy="0 0 0"/>
       <mass value="${chassisMass}"/>
       <xacro:box_inertia m="${chassisMass}" x="${chassisLength}" y="${chassisWidth}" z="${chassisHeight}"/>
@@ -135,5 +143,5 @@
       <parent link="zed2i_camera_link"/>
       <child link="base_link"/>
-      <origin xyz="-0.5 0 0.375" rpy="0 0 0"/>
+      <origin xyz="-0.35 0 -0.25" rpy="0 0 0"/>
     </joint>
   </xacro:if>
@@ -143,5 +151,5 @@
       <parent link="base_link"/>
       <child link="zed2i_camera_link"/>
-      <origin xyz="0.5 0 -0.375" rpy="0 0 0"/>
+      <origin xyz="0.35 0 0.25" rpy="0 0 0"/>
     </joint>
   </xacro:unless>
@@ -198,5 +206,5 @@
     <parent link="base_link"/>
     <child link="left_front"/>
-    <axis xyz="0.0 -1.0 0.0"/>
+    <axis xyz="0.0 1.0 0.0"/>
   </joint>
   <joint name="left_back_wheel" type="continuous">
@@ -204,5 +212,5 @@
     <parent link="base_link"/>
     <child link="left_back"/>
-    <axis xyz="0.0 -1.0 0.0"/>
+    <axis xyz="0.0 1.0 0.0"/>
   </joint>
   <joint name="right_back_wheel" type="continuous">

Commit message: Added proper measurements

File: src/robot_description/models/master_ASM/urdf/master_ASM.urdf.xacro (robot description, xacro)
@@ -2,11 +2,11 @@
 <robot name="Master_ASM" xmlns:xacro="http://www.ros.org/wiki/xacro">
   <xacro:property name="PI" value="3.1415926535897931"/>
-  <xacro:property name="chassisHeight" value="0.1"/>
-  <xacro:property name="chassisLength" value="0.8"/>
-  <xacro:property name="chassisWidth" value="0.5"/>
-  <xacro:property name="chassisMass" value="50"/>
-  <xacro:property name="wheelWidth" value="0.05"/>
-  <xacro:property name="wheelRadius" value="0.2"/>
-  <xacro:property name="wheelMass" value="5"/>
+  <xacro:property name="chassisHeight" value="0.64"/>
+  <xacro:property name="chassisLength" value="1.1"/>
+  <xacro:property name="chassisWidth" value="0.512"/>
+  <xacro:property name="chassisMass" value="55"/>
+  <xacro:property name="wheelWidth" value="0.11"/>
+  <xacro:property name="wheelRadius" value="0.15"/>
+  <xacro:property name="wheelMass" value="2"/>
   <xacro:macro name="box_inertia" params="m x y z">
     <inertia  ixx="${m*(y*y+z*z)/12}" ixy = "0" ixz = "0"

Commit message: begining tests

File: src/robot_description/models/master_ASM/urdf/master_ASM.urdf.xacro (robot description, xacro)
@@ -4,5 +4,5 @@
      Commit Version: 1.6.0-4-g7f85cfe  Build Version: 1.6.7995.38578
      For more information, please see http://wiki.ros.org/sw_urdf_exporter -->
-<robot name="Master_ASM" xmlns:xacro="http://www.ros.org/wiki/xacro">
+<robot name="Complicated" xmlns:xacro="http://www.ros.org/wiki/xacro">
   <link name="base_link">
     <origin xyz="0 0 0" rpy="0 0 0" />
@@ -53,14 +53,14 @@
   </link>
   <!-- ZED 2i Camera -->
-  <xacro:arg name="use_zed_localization" default="true" />
+  <!-- <xacro:arg name="use_zed_localization" default="true" />
   <xacro:include filename="$(find zed_wrapper)/urdf/zed_macro.urdf.xacro" />
-  <xacro:zed_camera name="zed2i" model="zed2i" enable_gnss="false">
+  <xacro:zed_camera name="zed2i" model="zed2i" enable_gnss="false"> -->
     <!-- This block is required even if enable_gnss="false" for some reason, but you can leave it empty -->
-    <gnss_origin></gnss_origin>
-  </xacro:zed_camera>
+    <!-- <gnss_origin></gnss_origin>
+  </xacro:zed_camera> -->
   <!-- Add a joint to connect the ZED 2i Camera model to the robot -->
-  <xacro:if value="$(arg use_zed_localization)">
+  <!-- <xacro:if value="$(arg use_zed_localization)"> -->
     <!-- ZED Localization -> The reference link is 'zed2i_camera_link' and 'base_link' is a child -->
-    <joint name="zed2i_joint" type="fixed">
+    <!-- <joint name="zed2i_joint" type="fixed">
       <parent link="zed2i_camera_link"/>
       <child link="base_link"/>
@@ -68,12 +68,12 @@
     </joint>
   </xacro:if>
-  <xacro:unless value="$(arg use_zed_localization)">
+  <xacro:unless value="$(arg use_zed_localization)"> -->
     <!-- NO ZED Localization -> 'zed2i_camera_link' is a child of 'base_link' -->
-    <joint name="zed2i_joint" type="fixed">
+    <!-- <joint name="zed2i_joint" type="fixed">
       <parent link="base_link"/>
       <child link="zed2i_camera_link"/>
       <origin xyz="0.5 0 -0.375" rpy="0 0 0"/>
     </joint>
-  </xacro:unless>
+  </xacro:unless> -->
   <gazebo reference="zed2i_camera_link">
     <sensor name="camera" type="camera">

Commit message: added muli-camera zed code

File: src/robot_description/models/master_ASM/urdf/master_ASM.urdf.xacro (robot description, xacro)
@@ -52,28 +52,45 @@
     </collision>
   </link>
-  <!-- ZED 2i Camera -->
+  <xacro:arg name="zed2i_front" />
+  <xacro:arg name="zed2i_rear" />
+  <xacro:arg name="zed2i" />
+  <xacro:arg name="zed2i" />
   <xacro:arg name="use_zed_localization" default="true" />
   <xacro:include filename="$(find zed_wrapper)/urdf/zed_macro.urdf.xacro" />
-  <xacro:zed_camera name="zed2i" model="zed2i" enable_gnss="false">
-    <!-- This block is required even if enable_gnss="false" for some reason, but you can leave it empty -->
-    <gnss_origin></gnss_origin>
-  </xacro:zed_camera>
-  <!-- Add a joint to connect the ZED 2i Camera model to the robot -->
+   <!-- Add the first ZED Camera -->
+  <xacro:zed_camera name="zed2i_front" model="zed2i" />
+  <!-- Add the second ZED Camera -->
+  <xacro:zed_camera name="zed2i_rear" model="zed2i" />
   <xacro:if value="$(arg use_zed_localization)">
-    <!-- ZED Localization -> The reference link is 'zed2i_camera_link' and 'base_link' is a child -->
-    <joint name="zed2i_joint" type="fixed">
-      <parent link="zed2i_camera_link"/>
+    <!-- ZED Localization -> The reference link is '$(arg camera_name_1)_camera_link' and 'base_link' is a child -->
+    <joint name="zed2i_front_joint" type="fixed">
+      <parent link="zed2i_front_camera_link"/>
       <child link="base_link"/>
-      <origin xyz="-0.5 0 0.375" rpy="0 0 0"/>
+      <origin
+        xyz="-0.12 0.0 -0.25"
+        rpy="0 0 0"
+      />
     </joint>
   </xacro:if>
   <xacro:unless value="$(arg use_zed_localization)">
-    <!-- NO ZED Localization -> 'zed2i_camera_link' is a child of 'base_link' -->
-    <joint name="zed2i_joint" type="fixed">
+    <!-- NO ZED Localization -> '$(arg camera_name)_camera_link' is a child of 'base_link' -->
+    <joint name="zed2i_front_joint" type="fixed">
       <parent link="base_link"/>
-      <child link="zed2i_camera_link"/>
-      <origin xyz="0.5 0 -0.375" rpy="0 0 0"/>
+      <child link="zed2i_front_camera_link"/>
+      <origin
+        xyz="0.12 0.0 0.25"
+        rpy="0 0 0"
+      />
     </joint>
   </xacro:unless>
+   <joint name="zed2i_rear_joint" type="fixed">
+    <parent link="base_link"/>
+    <child link="zed2i_rear_camera_link"/>
+    <origin
+      xyz="-0.12 0.0 0.25"
+      rpy="0 0 ${M_PI}"
+    />
+  </joint>
+  <!-- THIS STILL NEEDS TO CHANGE :)) -->
   <gazebo reference="zed2i_camera_link">
     <sensor name="camera" type="camera">

Commit message: renamed "zed_node_front" back to "zed_node" to maintain compatibility with single zed launch files.

File: src/robot_description/models/master_ASM/urdf/master_ASM.urdf.xacro (robot description, xacro)
@@ -55,15 +55,17 @@
   <xacro:include filename="$(find zed_wrapper)/urdf/zed_macro.urdf.xacro" />
    <!-- Add the first ZED Camera -->
-  <xacro:zed_camera name="zed2i_front" model="zed2i" enable_gnss="false">
+  <xacro:zed_camera name="zed2i" model="zed2i" enable_gnss="false">
     <!-- This block is required even if enable_gnss="false" for some reason, but you can leave it empty -->
     <gnss_origin></gnss_origin>
+  </xacro:zed_camera>
   <!-- Add the second ZED Camera -->
   <xacro:zed_camera name="zed2i_rear" model="zed2i" enable_gnss="false">
     <!-- This block is required even if enable_gnss="false" for some reason, but you can leave it empty -->
     <gnss_origin></gnss_origin>
+  </xacro:zed_camera>
   <xacro:if value="$(arg use_zed_localization)">
     <!-- ZED Localization -> The reference link is '$(arg camera_name_1)_camera_link' and 'base_link' is a child -->
-    <joint name="zed2i_front_joint" type="fixed">
-      <parent link="zed2i_front_camera_link"/>
+    <joint name="zed2i_joint" type="fixed">
+      <parent link="zed2i_camera_link"/>
       <child link="base_link"/>
       <origin
@@ -75,7 +77,7 @@
   <xacro:unless value="$(arg use_zed_localization)">
     <!-- NO ZED Localization -> '$(arg camera_name)_camera_link' is a child of 'base_link' -->
-    <joint name="zed2i_front_joint" type="fixed">
+    <joint name="zed2i_joint" type="fixed">
       <parent link="base_link"/>
-      <child link="zed2i_front_camera_link"/>
+      <child link="zed2i_camera_link"/>
       <origin
         xyz="0.12 0.0 0.25"
@@ -84,5 +86,5 @@
     </joint>
   </xacro:unless>
-   <joint name="zed2i_rear_joint" type="fixed">
+  <joint name="zed2i_rear_joint" type="fixed">
     <parent link="base_link"/>
     <child link="zed2i_rear_camera_link"/>
@@ -92,8 +94,6 @@
     />
   </joint>
-  <!-- THIS STILL NEEDS TO CHANGE :)) -->
   <gazebo reference="zed2i_camera_link">
     <sensor name="camera" type="camera">
-      <!-- <visualize>true</visualize> -->
       <always_on>true</always_on>
       <update_rate>30</update_rate>
@@ -115,5 +115,4 @@
     </sensor>
     <sensor name="depthcamera" type="depth">
-      <!-- <visualize>true</visualize> -->
       <always_on>true</always_on>
       <update_rate>30</update_rate>
@@ -135,4 +134,45 @@
     </sensor>
   </gazebo>
+  <!-- TODO: Test if this works in Gazebo (both ZEDs) -->
+  <!-- <gazebo reference="zed2i_rear_camera_link">
+    <sensor name="camera_rear" type="camera">
+      <always_on>true</always_on>
+      <update_rate>30</update_rate>
+      <camera>
+        <horizontal_fov>1.91986218</horizontal_fov>
+        <image>
+          <format>R8G8B8</format>
+          <width>1280</width>
+          <height>720</height>
+        </image>
+        <clip>
+          <near>0.3</near>
+          <far>5.0</far>
+        </clip>
+      </camera>
+      <topic>/color/image_rear</topic>
+      <info_topic>/color/camera_info_rear</info_topic>
+      <gz_frame_id>zed2i_rear_left_camera_optical_frame</gz_frame_id>
+    </sensor>
+    <sensor name="depthcamera_rear" type="depth">
+      <always_on>true</always_on>
+      <update_rate>30</update_rate>
+      <camera>
+        <horizontal_fov>1.91986218</horizontal_fov>
+        <image>
+          <format>R8G8B8</format>
+          <width>1280</width>
+          <height>720</height>
+        </image>
+        <clip>
+          <near>0.3</near>
+          <far>20.0</far>
+        </clip>
+      </camera>
+      <topic>/depth/image_rear</topic>
+      <info_topic>/depth/camera_info_rear</info_topic>
+      <gz_frame_id>zed2i_rear_left_camera_optical_frame</gz_frame_id>
+    </sensor>
+  </gazebo> -->
   <link
     name="swerve1_Link">

Commit message: small urdf changes

File: src/robot_description/models/master_ASM/urdf/master_ASM.urdf.xacro (robot description, xacro)
@@ -65,23 +65,17 @@
   </xacro:zed_camera>
   <xacro:if value="$(arg use_zed_localization)">
-    <!-- ZED Localization -> The reference link is '$(arg camera_name_1)_camera_link' and 'base_link' is a child -->
+    <!-- ZED Localization -> The reference link is 'zed2i_camera_link' and 'base_link' is a child -->
     <joint name="zed2i_joint" type="fixed">
       <parent link="zed2i_camera_link"/>
       <child link="base_link"/>
-      <origin
-        xyz="-0.12 0.0 -0.25"
-        rpy="0 0 0"
-      />
+      <origin xyz="-0.5 0 0.375" rpy="0 0 0"/>
     </joint>
   </xacro:if>
   <xacro:unless value="$(arg use_zed_localization)">
-    <!-- NO ZED Localization -> '$(arg camera_name)_camera_link' is a child of 'base_link' -->
+    <!-- NO ZED Localization -> 'zed2i_camera_link' is a child of 'base_link' -->
     <joint name="zed2i_joint" type="fixed">
       <parent link="base_link"/>
       <child link="zed2i_camera_link"/>
-      <origin
-        xyz="0.12 0.0 0.25"
-        rpy="0 0 0"
-      />
+      <origin xyz="0.5 0 -0.375" rpy="0 0 0"/>
     </joint>
   </xacro:unless>
@@ -89,8 +83,5 @@
     <parent link="base_link"/>
     <child link="zed2i_rear_camera_link"/>
-    <origin
-      xyz="-0.12 0.0 0.25"
-      rpy="0 0 ${M_PI}"
-    />
+    <origin xyz="0.5 0 -0.375" rpy="0 0 ${M_PI}"/>
   </joint>
   <gazebo reference="zed2i_camera_link">

Commit message: gazebo testing changes

File: src/robot_description/models/master_ASM/urdf/master_ASM.urdf.xacro (robot description, xacro)
@@ -83,5 +83,5 @@
     <parent link="base_link"/>
     <child link="zed2i_rear_camera_link"/>
-    <origin xyz="0.5 0 -0.375" rpy="0 0 ${M_PI}"/>
+    <origin xyz="-0.5 0 -0.375" rpy="0 0 ${M_PI}"/>
   </joint>
   <gazebo reference="zed2i_camera_link">
@@ -125,6 +125,5 @@
     </sensor>
   </gazebo>
-  <!-- TODO: Test if this works in Gazebo (both ZEDs) -->
-  <!-- <gazebo reference="zed2i_rear_camera_link">
+  <gazebo reference="zed2i_rear_camera_link">
     <sensor name="camera_rear" type="camera">
       <always_on>true</always_on>
@@ -165,5 +164,5 @@
       <gz_frame_id>zed2i_rear_left_camera_optical_frame</gz_frame_id>
     </sensor>
-  </gazebo> -->
+  </gazebo>
   <link
     name="swerve1_Link">
